File: Debug.kicad_sch (KiCad schematic)
At the start: 1 part, among them J3 Conn_02x07_Odd_Even

Commit message: t
Parts:
- removed J3: Conn_02x07_Odd_Even, symbol Connector_Generic:Conn_02x07_Odd_Even
Connections:
- no-connect marks 7 -> 0
Other:
- note removed: "PinHeader_2x07_P1.27mm_Vertical_SMD."

Commit message: Début Debug + MAJ MCU
Parts:
- added J2: Conn_02x10_Odd_Even, symbol Connector_Generic:Conn_02x10_Odd_Even
- added R18, R19, R20: 10K, symbol Device:R
Connections:
- new net: J2.17 (Pin_17), R19.1
- new net: J2.11 (Pin_11), R20.1
- new net: J2.19 (Pin_19), R18.1
- new net GND: J2.10 (Pin_10), J2.12 (Pin_12), J2.14 (Pin_14), J2.16 (Pin_16), J2.18 (Pin_18), J2.20 (Pin_20), J2.4 (Pin_4), J2.6 (Pin_6), J2.8 (Pin_8), R18.2, R19.2, R20.2
- new net JTDI: J2.5 (Pin_5)
- new net SWCLK: J2.7 (Pin_7)
- new net SWDIO: J2.9 (Pin_9)
- new net TDO: J2.13 (Pin_13)
- new net TRST: J2.15 (Pin_15)
- new net VCC_DEBUG: J2.1 (Pin_1), J2.2 (Pin_2)
- new net nRST: J2.3 (Pin_3)

Commit message: t
Other:
- note added: "ref jlc : C27985148 ou C3975190"
Changed lines of the file:
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@@
 	(generator_version "9.0")
 	(paper "A4")
+	(text "ref jlc : C27985148 ou C3975190"
+		(exclude_from_sim no)
+		(at 145.288 119.126 0)
+		(effects
+			(font
+				(size 1.27 1.27)
+			)
+		)
+	)
 	(junction
 		(at 157.48 90.17)

Commit message: Dernieres pour review
Parts:
- removed J2: Conn_02x10_Odd_Even, symbol Connector_Generic:Conn_02x10_Odd_Even
- removed R18, R19, R20: 10K, symbol Device:R
- added J3: Conn_02x07_Odd_Even, symbol Connector_Generic:Conn_02x07_Odd_Even
Connections:
- net GND: now also J3.11 (Pin_11), J3.5 (Pin_5), J3.7 (Pin_7)
- net SWCLK: now also J3.6 (Pin_6)
- net SWDIO: now also J3.4 (Pin_4)
- net nRST: now also J3.12 (Pin_12)
- new net +3.3V: J3.3 (Pin_3)
- new net RX: J3.14 (Pin_14)
- new net SW0: J3.8 (Pin_8)
- new net TX: J3.13 (Pin_13)
- no-connect marks 0 -> 4
Other:
- note added: "PinHeader_2x07_P1.27mm_Vertical_SMD."

Commit message: revue schema
Other:
- note added: "pas besoin de tx rx et swo"
Changed lines of the file:
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@@
+		)
+	)
+	(text "pas besoin de tx rx et swo\n\n\n\n"
+		(exclude_from_sim no)
+		(at 85.344 97.536 0)
+		(effects
+			(font
+				(size 1.27 1.27)
+				(color 255 0 0 1)
+			)
 		)
 	)

Commit message: premieres modif depuis la review
Connections:
- net RX: no longer names the net of J3.14 (Pin_14)
- net SW0: no longer names the net of J3.8 (Pin_8)
- net TX: no longer names the net of J3.13 (Pin_13)
- no-connect marks 4 -> 7
Other:
- note removed: "pas besoin de tx rx et swo"
- note removed: "ref jlc : C27985148 ou C3975190"
Changed lines of the file:
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@@
-		)
-	)
-	(text "ref jlc : C27985148 ou C3975190"
-		(exclude_from_sim no)
-		(at 145.288 119.126 0)
-		(effects
-			(font
-				(size 1.27 1.27)
-			)
-		)
-	)
-	(text "pas besoin de tx rx et swo\n\n\n\n"
-		(exclude_from_sim no)
-		(at 85.344 97.536 0)
-		(effects
-			(font
-				(size 1.27 1.27)
-				(color 255 0 0 1)
-			)
 		)
 	)
@@
 	)
 	(no_connect
+		(at 72.39 90.17)
+	)
+	(no_connect
 		(at 85.09 74.93)
+	)
+	(no_connect
+		(at 85.09 90.17)
 	)
 	(no_connect
@@
 	(no_connect
 		(at 72.39 85.09)
+	)
+	(no_connect
+		(at 85.09 82.55)
 	)
 	(wire
@@
 	(wire
 		(pts
-			(xy 85.09 82.55) (xy 90.17 82.55)
-		)
-		(stroke
-			(width 0)
-			(type default)
-		)
-	)
-	(wire
-		(pts
 			(xy 85.09 77.47) (xy 90.17 77.47)
 		)
@@
 	(wire
 		(pts
-			(xy 69.85 90.17) (xy 72.39 90.17)
-		)
-		(stroke
-			(width 0)
-			(type default)
-		)
-	)
-	(wire
-		(pts
 			(xy 72.39 82.55) (xy 64.77 82.55)
-		)
-		(stroke
-			(width 0)
-			(type default)
-		)
-	)
-	(wire
-		(pts
-			(xy 85.09 90.17) (xy 90.17 90.17)
 		)
 		(stroke
@@
 		)
 	)
-	(global_label "RX"
-		(shape input)
-		(at 90.17 90.17 0)
-		(fields_autoplaced yes)
-		(effects
-			(font
-				(size 1.27 1.27)
-			)
-			(justify left)
-		)
-		(property "Intersheetrefs" "${INTERSHEET_REFS}"
-			(at 95.6347 90.17 0)
-			(effects
-				(font
-					(size 1.27 1.27)
-				)
-				(justify left)
-				(hide yes)
-			)
-		)
-	)
 	(global_label "SWDIO"
 		(shape input)
@@
 		(property "Intersheetrefs" "${INTERSHEET_REFS}"
 			(at 99.0214 77.47 0)
-			(effects
-				(font
-					(size 1.27 1.27)
-				)
-				(justify left)
-				(hide yes)
-			)
-		)
-	)
-	(global_label "SW0"
-		(shape input)
-		(at 90.17 82.55 0)
-		(fields_autoplaced yes)
-		(effects
-			(font
-				(size 1.27 1.27)
-			)
-			(justify left)
-		)
-		(property "Intersheetrefs" "${INTERSHEET_REFS}"
-			(at 97.0256 82.55 0)
 			(effects
 				(font
@@
 				(hide yes)
 			)
-		)
-	)
-	(global_label "TX"
-		(shape input)
-		(at 69.85 90.17 180)
-		(fields_autoplaced yes)
-		(effects
-			(font
-				(size 1.27 1.27)
-			)
-			(justify right)
-		)
-		(property "Intersheetrefs" "${INTERSHEET_REFS}"
-			(at 64.6877 90.17 0)
-			(effects
-				(font
-					(size 1.27 1.27)
-				)
-				(justify right)
-				(hide yes)
-			)
