File: Connecteurs.kicad_sch (KiCad schematic)
At the start: 2 parts, among them J2 USB_C_Receptacle_PowerOnly_6P

Commit message: t
Parts:
- added R18, R7: 5,1k, symbol Device:R
Connections:
- net GND: now reaches J2.A12 (GND), J2.B12 (GND)
- net GND: now also R18.2, R7.2
- net at J2.A5 (CC1): now also R18.1
- net USB+: now reaches J2.A9 (VBUS), J2.B9 (VBUS)
- net at J2.B5 (CC2): now also R7.1

Commit message: t
Parts:
- added C31: 4,7nF 2kV X7R, symbol Device:C
- added C32: 10n, symbol Device:C
- added C33: 100nF, symbol Device:C
- added C34: 4,7u, symbol Device:C
- added D3: ESD5Z5V0, Diode_SMD:D_SOD-523, symbol Diode:ESD5Zxx
- added F1: C19712554, symbol Device:Fuse
- added F2: Fuse, symbol Device:Fuse
- added FB1: BLM18PG121SN1D, symbol Device:FerriteBead
- added J3: Conn_02x07_Odd_Even, symbol Connector_Generic:Conn_02x07_Odd_Even
- added R19: 1M, symbol Device:R
- added R20: 0, symbol Device:R
- BT1: value Battery_Cell -> BH-18650-4; LCSC (none) -> C49118399
Connections:
- net GND: now also C31.2, C32.2, C33.2, C34.2, D3.2 (A), J3.11 (Pin_11), J3.5 (Pin_5), J3.7 (Pin_7), R19.2, R20.2
- net USB+: now also F1.2; no longer J2.A9 (VBUS), J2.B9 (VBUS)
- net GND1: now reaches J2.S1 (SHIELD)
- net GND1: now also C31.1, R19.1, R20.1
- new net: C32.1, D3.1 (K), FB1.1, J2.A9 (VBUS), J2.B9 (VBUS)
- new net: C33.1, C34.1, F1.1, FB1.2
- new net +3.3V: J3.3 (Pin_3)
- new net SWCLK: J3.6 (Pin_6)
- new net SWDIO: J3.4 (Pin_4)
- new net nRST: J3.12 (Pin_12)
- no-connect marks 0 -> 7
Other:
- note added: "PinHeader_2x07_P1.27mm_Vertical_SMD."
- note added: "esd capa et fb proche du connecteur"
- moved on the sheet: BT1, J2, R18, R7

Commit message: t
Parts:
- R20: now not fitted; now left out of the parts list
Changed lines of the file:
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@@
 		(unit 1)
 		(exclude_from_sim no)
-		(in_bom yes)
+		(in_bom no)
 		(on_board yes)
-		(dnp no)
+		(dnp yes)
 		(fields_autoplaced yes)
 		(property "Reference" "R20"

Commit message: schema v1
Parts:
- added D7: ESD5Z5V0, Diode_SMD:D_SOD-523, symbol Diode:ESD5Zxx
- added Q7: AO3401A, Package_TO_SOT_SMD:SOT-23, symbol Transistor_FET:AO3401A
- added R25: 100k, symbol Device:R
- added TP32, TP33: TestPoint, symbol Connector:TestPoint
- F1: value C19712554 -> SCF6125F2A250V; LCSC (none) -> C19712554
- F2: value Fuse -> SCF6125F2A250V; LCSC (none) -> C19712554
Connections:
- net at F2.1: now also BT1.1 (+), D7.1 (K), TP32.1
- net at F2.2: now also Q7.3 (D)
- net at C32.1, D3.1 (K), FB1.1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: now also TP33.1
- net BAT+ renamed GNDA
- net GNDA: now also D7.2 (A), R25.2; no longer BT1.1 (+)
- net USB+ renamed VBUS
- new net: Q7.1 (G), R25.1
- new net +BATT: Q7.2 (S)
Other:
- moved on the sheet: BT1, J3

Commit message: Connecteurs + sourcing
Parts:
- C32: footprint (none) -> Capacitor_SMD:C_0603_1608Metric
- C33: footprint (none) -> Capacitor_SMD:C_0402_1005Metric
- C34: footprint (none) -> Capacitor_SMD:C_0805_2012Metric
- FB1: footprint (none) -> Inductor_SMD:L_0603_1608Metric
- J2: footprint (none) -> Composants_Perso:Connector_GT-USB-7002A
- J3: footprint (none) -> Composants_Perso:Connector_STLINKV3_Minie_14P
- R18, R19, R20, R25, R7: footprint (none) -> Resistor_SMD:R_0603_1608Metric
- TP32, TP33: footprint (none) -> TestPoint:TestPoint_Pad_D1.5mm
Connections:
- net +3.3V renamed +3V3
Other:
- note added: "PAS EN BASIC SUR JLCPCB"
- note added: "bidirectionnel"
- note added: "plutôt sur jlpcb C49118395"
- note removed: "PinHeader_2x07_P1.27mm_Vertical_SMD."
Changed lines of the file:
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@@
 		)
 	)
-	(text " PinHeader_2x07_P1.27mm_Vertical_SMD."
+	(text "PAS EN BASIC SUR JLCPCB"
 		(exclude_from_sim no)
-		(at 221.996 64.262 0)
+		(at 50.546 99.822 0)
 		(effects
 			(font
 				(size 1.27 1.27)
+				(color 255 16 22 1)
+			)
+		)
+	)
+	(text "plutôt sur jlpcb C49118395\n"
+		(exclude_from_sim no)
+		(at 92.71 104.394 0)
+		(effects
+			(font
+				(size 1.27 1.27)
+			)
+		)
+	)
+	(text "bidirectionnel\n"
+		(exclude_from_sim no)
+		(at 135.636 110.49 0)
+		(effects
+			(font
+				(size 1.27 1.27)
+				(color 255 0 4 1)
 			)
 		)
@@
 	(wire
 		(pts
+			(xy 29.21 172.72) (xy 29.21 180.34)
+		)
+		(stroke
+			(width 0)
+			(type default)
+		)
+	)
+	(wire
+		(pts
 			(xy 127 36.83) (xy 132.08 36.83)
 		)
@@
 			)
 		)
-		(property "Footprint" ""
+		(property "Footprint" "Inductor_SMD:L_0603_1608Metric"
 			(at 123.19 38.608 90)
 			(effects
@@
 	)
 	(symbol
+		(lib_id "power:PWR_FLAG")
+		(at 29.21 172.72 0)
+		(unit 1)
+		(exclude_from_sim no)
+		(in_bom yes)
+		(on_board yes)
+		(dnp no)
+		(fields_autoplaced yes)
+		(property "Reference" "#FLG07"
+			(at 29.21 170.815 0)
+			(effects
+				(font
+					(size 1.27 1.27)
+				)
+				(hide yes)
+			)
+		)
+		(property "Value" "PWR_FLAG"
+			(at 29.21 167.64 0)
+			(effects
+				(font
+					(size 1.27 1.27)
+				)
+			)
+		)
+		(property "Footprint" ""
+			(at 29.21 172.72 0)
+			(effects
+				(font
+					(size 1.27 1.27)
+				)
+				(hide yes)
+			)
+		)
+		(property "Datasheet" "~"
+			(at 29.21 172.72 0)
+			(effects
+				(font
+					(size 1.27 1.27)
+				)
+				(hide yes)
+			)
+		)
+		(property "Description" "Special symbol for telling ERC where power comes from"
+			(at 29.21 172.72 0)
+			(effects
+				(font
+					(size 1.27 1.27)
+				)
+				(hide yes)
+			)
+		)
+		(pin "1"
+		)
+		(instances
+			(project ""
+				(path "/90bd0b60-6e70-43e1-8410-99fb54688c17/acdb258c-42de-401c-9111-59e7e388a012"
+					(reference "#FLG07")
+					(unit 1)
+				)
+			)
+		)
+	)
+	(symbol
 		(lib_id "power:VBUS")
 		(at 168.91 33.02 0)
@@
 			)
 		)
-		(property "Footprint" ""
+		(property "Footprint" "Resistor_SMD:R_0603_1608Metric"
 			(at 73.152 57.15 90)
 			(effects
@@
 			)
 		)
-		(property "Footprint" ""
+		(property "Footprint" "Resistor_SMD:R_0603_1608Metric"
 			(at 36.83 81.788 90)
 			(effects
@@
 			)
 		)
-		(property "Footprint" ""
+		(property "Footprint" "TestPoint:TestPoint_Pad_D1.5mm"
 			(at 78.74 36.83 0)
 			(effects
@@
 			)
 		)
-		(property "Footprint" ""
+		(property "Footprint" "Composants_Perso:Connector_STLINKV3_Minie_14P"
 			(at 219.71 44.45 0)
 			(effects
@@
 			)
 		)
-		(property "Footprint" ""
+		(property "Footprint" "Composants_Perso:Connector_GT-USB-7002A"
 			(at 60.96 41.91 0)
 			(effects
@@
 			)
 		)
-		(property "Footprint" ""
+		(property "Footprint" "TestPoint:TestPoint_Pad_D1.5mm"
 			(at 111.76 97.79 0)
 			(effects
@@
 			)
 		)
-		(property "Footprint" ""
+		(property "Footprint" "Capacitor_SMD:C_0603_1608Metric"
 			(at 113.9952 46.99 0)
 			(effects
@@
 			)
 		)
-		(property "Footprint" ""
+		(property "Footprint" "Resistor_SMD:R_0603_1608Metric"
 			(at 80.772 54.61 90)
 			(effects
@@
 			)
 		)
-		(property "Value" "+3.3V"
+		(property "Value" "+3V3"
 			(at 204.47 39.3699 90)
 			(effects
@@
 			)
 		)
-		(property "Footprint" ""
+		(property "Footprint" "Resistor_SMD:R_0603_1608Metric"
 			(at 153.162 110.49 90)
 			(effects
@@
 			)
 		)
-		(property "Footprint" ""
+		(property "Footprint" "Capacitor_SMD:C_0402_1005Metric"
 			(at 133.0452 46.99 0)
 			(effects
@@
 			)
 		)
-		(property "Footprint" ""
+		(property "Footprint" "Resistor_SMD:R_0603_1608Metric"
 			(at 36.83 91.948 90)
 			(effects
@@
 	)
 	(symbol
+		(lib_id "power:GND1")
+		(at 29.21 180.34 0)
+		(unit 1)
+		(exclude_from_sim no)
+		(in_bom yes)
+		(on_board yes)
+		(dnp no)
+		(fields_autoplaced yes)
+		(property "Reference" "#PWR065"
+			(at 29.21 186.69 0)
+			(effects
+				(font
+					(size 1.27 1.27)
+				)
+				(hide yes)
+			)
+		)
+		(property "Value" "GND1"
+			(at 29.21 185.42 0)
+			(effects
+				(font
+					(size 1.27 1.27)
+				)
+			)
+		)
+		(property "Footprint" ""
+			(at 29.21 180.34 0)
+			(effects
+				(font
+					(size 1.27 1.27)
+				)
+				(hide yes)
+			)
+		)
+		(property "Datasheet" ""
+			(at 29.21 180.34 0)
+			(effects
+				(font
+					(size 1.27 1.27)
+				)
+				(hide yes)
+			)
+		)
+		(property "Description" "Power symbol creates a global label with name \"GND1\" , ground"
+			(at 29.21 180.34 0)
+			(effects
+				(font
+					(size 1.27 1.27)
+				)
+				(hide yes)
+			)
+		)
+		(pin "1"
+		)
+		(instances
+			(project "Station_Meteo_pcb"
+				(path "/90bd0b60-6e70-43e1-8410-99fb54688c17/acdb258c-42de-401c-9111-59e7e388a012"
+					(reference "#PWR065")
+					(unit 1)
+				)
+			)
+		)
+	)
+	(symbol
 		(lib_id "Device:C")
 		(at 144.78 43.18 0)
@@
 			)
 		)
-		(property "Footprint" ""
+		(property "Footprint" "Capacitor_SMD:C_0805_2012Metric"
 			(at 145.7452 46.99 0)
 			(effects
