File: Connecteurs.kicad_sch (KiCad schematic)
At the start: 22 parts, among them J10 Conn_01x02_Pin, J11 Conn_01x02_Pin, J2 USB_C_Receptacle_PowerOnly_6P, J3 Conn_02x07_Odd_Even, Q7 AO3401A

Commit message: t
Parts:
- BT1: footprint (none) -> Composants_Perso:BH-18650-4
- J2: footprint Composants_Perso:Connector_GT-USB-7002A -> Composants_Perso:UC18-0B06F68011; LCSC (none) -> C963365
- J3: LCSC (none) -> C42462827
Changed lines of the file:
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@@
 			)
 		)
-		(property "LCSC" ""
+		(property "LCSC" "C42462827"
 			(at 219.71 44.45 0)
 			(effects
@@
 			)
 		)
-		(property "Footprint" "Composants_Perso:Connector_GT-USB-7002A"
+		(property "Footprint" "Composants_Perso:UC18-0B06F68011"
 			(at 60.96 41.91 0)
 			(effects
@@
 			)
 		)
-		(property "LCSC" ""
+		(property "LCSC" "C963365"
 			(at 57.15 44.45 0)
 			(effects
@@
 			)
 		)
-		(property "Footprint" ""
+		(property "Footprint" "Composants_Perso:BH-18650-4"
 			(at 106.68 106.426 90)
 			(effects

Commit message: t
Parts:
- C31: value 4,7nF 2kV X7R -> 1nF 2kV X7R; footprint (none) -> Capacitor_SMD:C_1206_3216Metric; LCSC (none) -> C9196
- F1, F2: footprint (none) -> Composants_Perso:SCF6125F2A250V
Connections:
- net at J11.2 (Pin_2), Q7.2 (S): now also BT1.1 (+), D7.1 (K), F2.1, F2.2, Q7.3 (D), TP32.1
Other:
- note removed: "PAS EN BASIC SUR JLCPCB"
- note removed: "bidirectionnel"
- moved on the sheet: D7, F2, J11, Q7, R25

Commit message: t
Parts:
- C32: LCSC (none) -> C57112
- C33: value 100nF -> 100n; LCSC (none) -> C1525
- C34: value 4,7u -> 4.7u/25V; LCSC (none) -> C1779
- D3, D7: LCSC (none) -> C21714169
- FB1: LCSC (none) -> C14709
- J10, J11: value Conn_01x02_Pin -> DZ254S-11-02-48; LCSC (none) -> C5160785
- J2: value USB_C_Receptacle_PowerOnly_6P -> GT-USB-7002A
- J3: value Conn_02x07_Odd_Even -> BH127VS-14P-H49
- Q7: LCSC (none) -> C15127
- R18, R7: value 5,1k -> 5k1; LCSC (none) -> C23186
- R19: LCSC (none) -> C22935
- R25: LCSC (none) -> C25803
- TP32, TP33: now left out of the parts list

Commit message: t
Parts:
- J2: value GT-USB-7002A -> UC18-0B06F68011; LCSC C963365 -> C36936555
Connections:
- net at D7.1 (K), F2.2, J11.2 (Pin_2)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: no longer BT1.1 (+), F2.1, TP32.1
- new net: BT1.1 (+), F2.1, TP32.1
Changed lines of the file:
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@@
-	)
-	(junction
-		(at 118.11 97.79)
-		(diameter 0)
-		(color 0 0 0 0)
 	)
 	(junction
@@
 	)
 	(junction
-		(at 125.73 97.79)
-		(diameter 0)
-		(color 0 0 0 0)
-	)
-	(junction
 		(at 44.45 101.6)
 		(diameter 0)
@@
 		(pts
 			(xy 166.37 92.71) (xy 166.37 97.79)
-		)
-		(stroke
-			(width 0)
-			(type default)
-		)
-	)
-	(wire
-		(pts
-			(xy 125.73 97.79) (xy 118.11 97.79)
 		)
 		(stroke
@@
 			)
 		)
-		(property "Value" "GT-USB-7002A"
+		(property "Value" "UC18-0B06F68011"
 			(at 57.15 29.21 0)
 			(effects
@@
 			)
 		)
-		(property "LCSC" "C963365"
+		(property "LCSC" "C36936555"
 			(at 57.15 44.45 0)
 			(effects

Commit message: V1 Placement + Routage
Connections:
- net at D7.1 (K), J11.2 (Pin_2), Q7.2 (S): no longer F2.2, Q7.3 (D)
- new net: F2.2, Q7.3 (D)
Changed lines of the file:
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@@
-	)
-	(junction
-		(at 144.78 97.79)
-		(diameter 0)
-		(color 0 0 0 0)
 	)
 	(junction
@@
 	)
 	(junction
+		(at 149.86 97.79)
+		(diameter 0)
+		(color 0 0 0 0)
+	)
+	(junction
 		(at 44.45 101.6)
 		(diameter 0)
@@
 	)
 	(junction
-		(at 149.86 97.79)
-		(diameter 0)
-		(color 0 0 0 0)
-	)
-	(junction
-		(at 134.62 97.79)
-		(diameter 0)
-		(color 0 0 0 0)
-	)
-	(junction
 		(at 106.68 97.79)
 		(diameter 0)
@@
 	(wire
 		(pts
-			(xy 144.78 97.79) (xy 134.62 97.79)
-		)
-		(stroke
-			(width 0)
-			(type default)
-		)
-	)
-	(wire
-		(pts
 			(xy 180.34 36.83) (xy 180.34 33.02)
 		)
@@
 	(wire
 		(pts
-			(xy 149.86 97.79) (xy 144.78 97.79)
-		)
-		(stroke
-			(width 0)
-			(type default)
-		)
-	)
-	(wire
-		(pts
 			(xy 29.21 80.01) (xy 33.02 80.01)
 		)
@@
 	(wire
 		(pts
+			(xy 144.78 97.79) (xy 149.86 97.79)
+		)
+		(stroke
+			(width 0)
+			(type default)
+		)
+	)
+	(wire
+		(pts
 			(xy 214.63 41.91) (xy 207.01 41.91)
 		)
@@
 	(wire
 		(pts
+			(xy 125.73 97.79) (xy 134.62 97.79)
+		)
+		(stroke
+			(width 0)
+			(type default)
+		)
+	)
+	(wire
+		(pts
 			(xy 72.39 36.83) (xy 73.66 36.83)
 		)
 		(stroke
-			(width 0)
-			(type default)
-		)
-	)
-	(wire
-		(pts
-			(xy 125.73 97.79) (xy 134.62 97.79)
-		)
-		(stroke

Commit message: Placement + routage V2
Parts:
- renumbered TP32 to BAT+1, TP33 to VBUS1
Changed lines of the file:
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@@
 		(on_board yes)
 		(dnp no)
-		(property "Reference" "TP33"
+		(property "Reference" "VBUS1"
 			(at 72.136 30.988 0)
 			(effects
@@
 			(project "Station_Meteo_pcb"
 				(path "/90bd0b60-6e70-43e1-8410-99fb54688c17/acdb258c-42de-401c-9111-59e7e388a012"
-					(reference "TP33")
+					(reference "VBUS1")
 					(unit 1)
 				)
@@
 		(on_board yes)
 		(dnp no)
-		(property "Reference" "TP32"
+		(property "Reference" "BAT+1"
 			(at 105.156 91.948 0)
 			(effects
@@
 			(project "Station_Meteo_pcb"
 				(path "/90bd0b60-6e70-43e1-8410-99fb54688c17/acdb258c-42de-401c-9111-59e7e388a012"
-					(reference "TP32")
+					(reference "BAT+1")
 					(unit 1)
 				)
