File: Connecteurs.kicad_sch (KiCad schematic)
At the start: 22 parts, among them J10 DZ254S-11-02-48, J11 DZ254S-11-02-48, J2 UC18-0B06F68011, J3 BH127VS-14P-H49, Q7 AO3401A

Commit message: last push
Parts:
- BT1: LCSC C49118399 -> C7525438
Other:
- note removed: "plutôt sur jlpcb C49118395"
Changed lines of the file:
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@@
 		)
 	)
-	(text "plutôt sur jlpcb C49118395\n"
-		(exclude_from_sim no)
-		(at 92.71 104.394 0)
-		(effects
-			(font
-				(size 1.27 1.27)
-			)
-		)
-	)
 	(junction
 		(at 29.21 90.17)
@@
 			)
 		)
-		(property "LCSC" "C49118399"
+		(property "LCSC" "C7525438"
 			(at 106.68 107.95 0)
 			(effects
