File: Ecran.kicad_sch (KiCad schematic)
At the start: 18 parts, among them J1 Conn_01x24_Pin, Q1 Q_NMOS_GSD

Commit message: t
Parts:
- removed D1, D2, D3: MBR0530, Diode_SMD:D_SOD-123, symbol Diode:MBR0530
- added D1, D2, D8: 1N5819WS, Diode_SMD:D_SOD-323, symbol Diode:1N5819WS
Connections:
- net GND: now also D8.1 (K)
- net VGH: now also D1.1 (K)
- net VGL: now also D2.2 (A)
- net at C3.2, L1.2, Q1.3 (D): now also D1.2 (A)
- net at C3.1: now also D2.1 (K), D8.2 (A)

Commit message: schema v1
Parts:
- removed Q1: Q_NMOS_GSD, symbol Transistor_FET:Q_NMOS_GSD
- added Q1, Q2: AO3400A, Package_TO_SOT_SMD:SOT-23, symbol Transistor_FET:AO3400A
- added Q3: AO3401A, Package_TO_SOT_SMD:SOT-23, symbol Transistor_FET:AO3401A
- added R28: 0, symbol Device:R
- added R8, R9: 1M, symbol Device:R
- added TP27, TP28, TP29, TP30, TP31: TestPoint, symbol Connector:TestPoint
Connections:
- net GDR: now also Q1.1 (G), TP29.1
- net GND: now also Q2.2 (S), R9.2
- net RESE: now also Q1.2 (S), TP28.1
- net at C3.2, D1.2 (A), L1.2: now also Q1.3 (D), TP31.1
- net at C3.1, D2.1 (K), D8.2 (A): now also TP30.1
- net 3V3_OUT renamed EPD_PWR
- net EPD_PWR: now also R28.2, TP27.1
- new net: Q2.3 (D), Q3.1 (G), R8.2
- new net: Q3.3 (D), R28.1
- new net +3V3: Q3.2 (S), R8.1
- new net CMD_ALIM_SCREEN: Q2.1 (G), R9.1
Other:
- note added: "Alimenation écran"
- moved on the sheet: C10, C11, C12, C14, C3, C4, C6, C7, C8, C9, D1, D2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

Commit message: Connecteurs + sourcing
Parts:
- removed R28: 0, symbol Device:R
- added J12: Conn_01x02_Pin, Connector_PinHeader_2.54mm:PinHeader_1x02_P2.54mm_Vertical_SMD_Pin1Left, symbol Connector:Conn_01x02_Pin
- added R36: 1, Resistor_SMD:R_0603_1608Metric, symbol Device:R
- C10, C11, C14, C6, C7, C8, C9: footprint (none) -> Capacitor_SMD:C_0603_1608Metric; LCSC (none) -> C15849
- C12: footprint (none) -> Capacitor_SMD:C_0603_1608Metric
- C3, C4: footprint (none) -> Capacitor_SMD:C_0805_2012Metric
- J1: footprint (none) -> Composants_Perso:Connector_24P_epaper
- L1: footprint (none) -> Inductor_SMD:L_0805_2012Metric
- R3: value 3 -> 2; footprint (none) -> Resistor_SMD:R_0603_1608Metric
- R4, R8, R9: footprint (none) -> Resistor_SMD:R_0603_1608Metric
- TP27, TP28, TP29, TP30, TP31: footprint (none) -> TestPoint:TestPoint_Pad_D1.5mm
Connections:
- net EPD_PWR: now also J12.2 (Pin_2)
- net GND: now also R36.1; no longer R3.1
- net at Q3.3 (D): now also J12.1 (Pin_1)
- new net: R3.1, R36.2
Other:
- moved on the sheet: R3, TP28
