File: Ecran.kicad_sch (KiCad schematic)
At the start: 29 parts, among them J1 Conn_01x24_Pin, J6 DZ254S-11-02-48, Q1 AO3400A, Q2 AO3400A, Q3 AO3401A

Commit message: t
Parts:
- J1: LCSC (none) -> C7419878
Changed lines of the file:
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@@
 					(size 1.27 1.27)
 				)
+				(hide yes)
 			)
 		)
@@
 			)
 		)
-		(property "LCSC" ""
+		(property "LCSC" "C7419878"
 			(at 200.66 60.96 0)
 			(effects

Commit message: t
Parts:
- C10, C11, C14, C6, C7, C8, C9: value 1uF/50V -> 1u/50V
- C12: value 1uF/50V -> 1u/50V; LCSC (none) -> C15849
- C3, C4: value 4.7uF/25V -> 4.7u/25V; LCSC (none) -> C1779
- J1: value Conn_01x24_Pin -> ZX-FPC-FWSX0.5PH224
- L1: LCSC (none) -> C1046
- Q1, Q2: LCSC (none) -> C20917
- Q3: LCSC (none) -> C15127
- R3: LCSC (none) -> C22977
- R36: LCSC (none) -> C22936
- R4: value 10K -> 10k; LCSC (none) -> C25804
- R8, R9: LCSC (none) -> C22935
- TP27, TP28, TP29, TP30, TP31: now left out of the parts list

Commit message: t
Connections:
- net CMD_ALIM_SCREEN is gone; now on net EPD_PWR: Q2.1 (G), R9.1
- net EPD_PWR: no longer C4.2, C6.1, J1.15 (Pin_15), J1.16 (Pin_16), J6.2 (Pin_2), L1.1, TP27.1
- new net ALIM_SCREEN: C4.2, C6.1, J1.15 (Pin_15), J1.16 (Pin_16), J6.2 (Pin_2), L1.1, TP27.1
Other:
- moved on the sheet: R9, TP27
Changed lines of the file:
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@@
 	)
 	(junction
+		(at 96.52 74.93)
+		(diameter 0)
+		(color 0 0 0 0)
+	)
+	(junction
 		(at 207.01 68.58)
 		(diameter 0)
@@
 	)
 	(junction
-		(at 100.33 74.93)
-		(diameter 0)
-		(color 0 0 0 0)
-	)
-	(junction
 		(at 264.16 73.66)
 		(diameter 0)
@@
 	(wire
 		(pts
-			(xy 149.86 72.39) (xy 149.86 73.66)
+			(xy 149.86 67.31) (xy 149.86 73.66)
 		)
 		(stroke
@@
 	(wire
 		(pts
-			(xy 93.98 74.93) (xy 100.33 74.93)
+			(xy 53.34 81.28) (xy 59.69 81.28)
+		)
+		(stroke
+			(width 0)
+			(type default)
+		)
+	)
+	(wire
+		(pts
+			(xy 93.98 74.93) (xy 96.52 74.93)
 		)
 		(stroke
@@
 	(wire
 		(pts
-			(xy 59.69 88.9) (xy 59.69 91.44)
+			(xy 59.69 90.17) (xy 59.69 91.44)
+		)
+		(stroke
+			(width 0)
+			(type default)
+		)
+	)
+	(wire
+		(pts
+			(xy 96.52 74.93) (xy 100.33 74.93)
 		)
 		(stroke
@@
 	(wire
 		(pts
+			(xy 59.69 82.55) (xy 59.69 81.28)
+		)
+		(stroke
+			(width 0)
+			(type default)
+		)
+	)
+	(wire
+		(pts
 			(xy 205.74 68.58) (xy 207.01 68.58)
 		)
@@
 	(wire
 		(pts
-			(xy 100.33 74.93) (xy 102.87 74.93)
-		)
-		(stroke
-			(width 0)
-			(type default)
-		)
-	)
-	(wire
-		(pts
 			(xy 262.89 91.44) (xy 264.16 91.44)
 		)
@@
 		)
 	)
-	(wire
-		(pts
-			(xy 55.88 81.28) (xy 59.69 81.28)
-		)
-		(stroke
-			(width 0)
-			(type default)
-		)
-	)
-	(global_label "CMD_ALIM_SCREEN"
-		(shape input)
-		(at 55.88 81.28 180)
-		(fields_autoplaced yes)
-		(effects
-			(font
-				(size 1.27 1.27)
-			)
-			(justify right)
-		)
-		(property "Intersheetrefs" "${INTERSHEET_REFS}"
-			(at 35.4173 81.28 0)
-			(effects
-				(font
-					(size 1.27 1.27)
-				)
-				(justify right)
-				(hide yes)
-			)
-		)
-	)
 	(global_label "VGL"
 		(shape input)
@@
 	(global_label "EPD_PWR"
 		(shape input)
-		(at 102.87 74.93 0)
+		(at 53.34 81.28 180)
 		(fields_autoplaced yes)
 		(effects
@@
 				(size 1.27 1.27)
 			)
-			(justify left)
+			(justify right)
 		)
 		(property "Intersheetrefs" "${INTERSHEET_REFS}"
-			(at 114.5032 74.93 0)
+			(at 41.7068 81.28 0)
 			(effects
 				(font
 					(size 1.27 1.27)
 				)
-				(justify left)
+				(justify right)
 				(hide yes)
 			)
@@
 		)
 	)
+	(global_label "ALIM_SCREEN"
+		(shape input)
+		(at 100.33 74.93 0)
+		(fields_autoplaced yes)
+		(effects
+			(font
+				(size 1.27 1.27)
+			)
+			(justify left)
+		)
+		(property "Intersheetrefs" "${INTERSHEET_REFS}"
+			(at 115.8337 74.93 0)
+			(effects
+				(font
+					(size 1.27 1.27)
+				)
+				(justify left)
+				(hide yes)
+			)
+		)
+	)
 	(global_label "RESE"
 		(shape input)
@@
 		)
 	)
-	(global_label "EPD_PWR"
+	(global_label "ALIM_SCREEN"
 		(shape input)
 		(at 207.01 96.52 270)
@@
 		)
 		(property "Intersheetrefs" "${INTERSHEET_REFS}"
-			(at 207.01 108.1532 90)
+			(at 207.01 112.0237 90)
 			(effects
 				(font
@@
 		)
 	)
-	(global_label "EPD_PWR"
+	(global_label "ALIM_SCREEN"
 		(shape input)
-		(at 149.86 72.39 90)
+		(at 149.86 67.31 180)
 		(fields_autoplaced yes)
 		(effects
@@
 				(size 1.27 1.27)
 			)
-			(justify left)
+			(justify right)
 		)
 		(property "Intersheetrefs" "${INTERSHEET_REFS}"
-			(at 149.86 60.7568 90)
+			(at 134.3563 67.31 0)
 			(effects
 				(font
 					(size 1.27 1.27)
 				)
-				(justify left)
+				(justify right)
 				(hide yes)
 			)
@@
 		(on_board yes)
 		(dnp no)
-		(fields_autoplaced yes)
 		(property "Reference" "C4"
-			(at 137.16 66.04 90)
+			(at 133.858 75.946 90)
 			(effects
 				(font
@@
 		)
 		(property "Value" "4.7u/25V"
-			(at 137.16 68.58 90)
+			(at 133.858 78.486 90)
 			(effects
 				(font
@@
 	(symbol
 		(lib_id "Connector:TestPoint")
-		(at 100.33 74.93 0)
+		(at 96.52 74.93 0)
 		(unit 1)
 		(exclude_from_sim no)
@@
 		(dnp no)
 		(property "Reference" "TP27"
-			(at 98.298 69.342 0)
+			(at 94.488 69.342 0)
 			(effects
 				(font
@@
 		)
 		(property "Value" "TestPoint"
-			(at 88.9 71.374 0)
+			(at 85.09 71.374 0)
 			(effects
 				(font
@@
 		)
 		(property "Footprint" "TestPoint:TestPoint_Pad_D1.5mm"
-			(at 105.41 74.93 0)
+			(at 101.6 74.93 0)
 			(effects
 				(font
@@
 		)
 		(property "Datasheet" "~"
-			(at 105.41 74.93 0)
+			(at 101.6 74.93 0)
 			(effects
 				(font
@@
 		)
 		(property "Description" "test point"
-			(at 100.33 74.93 0)
+			(at 96.52 74.93 0)
 			(effects
 				(font
@@
 		)
 		(property "LCSC" ""
-			(at 100.33 74.93 0)
+			(at 96.52 74.93 0)
 			(effects
 				(font
@@
 		)
 		(property "Arrow Part Number" ""
-			(at 100.33 74.93 0)
+			(at 96.52 74.93 0)
 			(effects
 				(font
@@
 		)
 		(property "Arrow Price/Stock" ""
-			(at 100.33 74.93 0)
+			(at 96.52 74.93 0)
 			(effects
 				(font
@@
 		)
 		(property "Height" ""
-			(at 100.33 74.93 0)
+			(at 96.52 74.93 0)
 			(effects
 				(font
@@
 		)
 		(property "Manufacturer_Name" ""
-			(at 100.33 74.93 0)
+			(at 96.52 74.93 0)
 			(effects
 				(font
@@
 		)
 		(property "Manufacturer_Part_Number" ""
-			(at 100.33 74.93 0)
+			(at 96.52 74.93 0)
 			(effects
 				(font
@@
 		)
 		(property "Mouser Part Number" ""
-			(at 100.33 74.93 0)
+			(at 96.52 74.93 0)
 			(effects
 				(font
@@
 		)
 		(property "Mouser Price/Stock" ""
-			(at 100.33 74.93 0)
+			(at 96.52 74.93 0)
 			(effects
 				(font
@@
 	(symbol
 		(lib_id "Device:R")
-		(at 59.69 85.09 0)
+		(at 59.69 86.36 0)
 		(unit 1)
 		(exclude_from_sim no)
@@
 		(fields_autoplaced yes)
 		(property "Reference" "R9"
-			(at 62.23 83.8199 0)
+			(at 62.23 85.0899 0)
 			(effects
 				(font
@@
 		)
 		(property "Value" "1M"
-			(at 62.23 86.3599 0)
+			(at 62.23 87.6299 0)
 			(effects
 				(font
@@
 		)
 		(property "Footprint" "Resistor_SMD:R_0603_1608Metric"
-			(at 57.912 85.09 90)
+			(at 57.912 86.36 90)
 			(effects
 				(font
@@
 		)
 		(property "Datasheet" "~"
-			(at 59.69 85.09 0)
+			(at 59.69 86.36 0)
 			(effects
 				(font
@@
 		)
 		(property "Description" "Resistor"
-			(at 59.69 85.09 0)
+			(at 59.69 86.36 0)
 			(effects
 				(font
@@
 		)
 		(property "LCSC" "C22935"
-			(at 59.69 85.09 0)
+			(at 59.69 86.36 0)
 			(effects
 				(font
@@
 		)
 		(property "Arrow Part Number" ""
-			(at 59.69 85.09 0)
+			(at 59.69 86.36 0)
 			(effects
 				(font
@@
 		)
 		(property "Arrow Price/Stock" ""
-			(at 59.69 85.09 0)
+			(at 59.69 86.36 0)
 			(effects
 				(font
@@
 		)
 		(property "Height" ""
-			(at 59.69 85.09 0)
+			(at 59.69 86.36 0)
 			(effects
 				(font
@@
 		)
 		(property "Manufacturer_Name" ""
-			(at 59.69 85.09 0)
+			(at 59.69 86.36 0)
 			(effects
 				(font
@@
 		)
 		(property "Manufacturer_Part_Number" ""
-			(at 59.69 85.09 0)
+			(at 59.69 86.36 0)
 			(effects
 				(font
@@
 		)
 		(property "Mouser Part Number" ""
-			(at 59.69 85.09 0)
+			(at 59.69 86.36 0)
 			(effects
 				(font
@@
 		)
 		(property "Mouser Price/Stock" ""
-			(at 59.69 85.09 0)
+			(at 59.69 86.36 0)
 			(effects
 				(font

Commit message: Placement + routage V2
Parts:
- renumbered TP27 to ALIM_S1, TP29 to GDR, TP28 to RESE1
Changed lines of the file:
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@@
 		(on_board yes)
 		(dnp no)
-		(property "Reference" "TP29"
+		(property "Reference" "GDR"
 			(at 142.748 54.102 0)
 			(effects
@@
 			(project "Station_Meteo_pcb"
 				(path "/90bd0b60-6e70-43e1-8410-99fb54688c17/3922ef04-1be0-4a1a-a432-baea08402c76"
-					(reference "TP29")
+					(reference "GDR")
 					(unit 1)
 				)
@@
 		(on_board yes)
 		(dnp no)
-		(property "Reference" "TP27"
+		(property "Reference" "ALIM_S1"
 			(at 94.488 69.342 0)
 			(effects
@@
 			(project "Station_Meteo_pcb"
 				(path "/90bd0b60-6e70-43e1-8410-99fb54688c17/3922ef04-1be0-4a1a-a432-baea08402c76"
-					(reference "TP27")
+					(reference "ALIM_S1")
 					(unit 1)
 				)
@@
 		(on_board yes)
 		(dnp no)
-		(property "Reference" "TP28"
+		(property "Reference" "RESE1"
 			(at 154.178 42.672 0)
 			(effects
@@
 			(project "Station_Meteo_pcb"
 				(path "/90bd0b60-6e70-43e1-8410-99fb54688c17/3922ef04-1be0-4a1a-a432-baea08402c76"
-					(reference "TP28")
+					(reference "RESE1")
 					(unit 1)
 				)

Commit message: t
Parts:
- renumbered GDR to GDR1
Changed lines of the file:
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@@
 		(on_board yes)
 		(dnp no)
-		(property "Reference" "GDR"
+		(property "Reference" "GDR1"
 			(at 142.748 54.102 0)
 			(effects
@@
 			(project "Station_Meteo_pcb"
 				(path "/90bd0b60-6e70-43e1-8410-99fb54688c17/3922ef04-1be0-4a1a-a432-baea08402c76"
-					(reference "GDR")
+					(reference "GDR1")
 					(unit 1)
 				)

Commit message: Suite DRC
Parts:
- J1: footprint Composants_Perso:Connector_24P_epaper -> Composants_Perso:Connector_1x24_epaper
Changed lines of the file:
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@@
 			)
 		)
-		(property "Footprint" "Composants_Perso:Connector_24P_epaper"
+		(property "Footprint" "Composants_Perso:Connector_1x24_epaper"
 			(at 200.66 60.96 0)
 			(effects

Commit message: modif pour commande
Parts:
- J6: footprint Connector_PinHeader_2.54mm:PinHeader_1x02_P2.54mm_Vertical_SMD_Pin1Right -> Connector_PinHeader_2.54mm:PinHeader_1x02_P2.54mm_Vertical_SMD_Pin1Left
Changed lines of the file:
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@@
 			)
 		)
-		(property "Footprint" "Connector_PinHeader_2.54mm:PinHeader_1x02_P2.54mm_Vertical_SMD_Pin1Right"
+		(property "Footprint" "Connector_PinHeader_2.54mm:PinHeader_1x02_P2.54mm_Vertical_SMD_Pin1Left"
 			(at 91.44 80.01 0)
 			(effects
