File: Alimentation.kicad_sch (KiCad schematic)
At the start: 34 parts, among them IC1 DW01S, Q2 PMOS, Q3 NMOS, Q4 PMOS, Q5 FS8205A, Q6 NMOS, Q8 PMOS, U3 TP4056-42-ESOP8, U4 TPS63802DLAR

Commit message: t
Connections:
- net OUT- is gone; now on net GND: C16.2, C18.2, C29.1, Q5.6, Q5.7, R15.2, R17.2, U3.1 (TEMP), U3.3 (GND), U3.9 (EPAD)
- net BAT-: now also Q5.2, Q5.3; no longer Q5.5
- new net: IC1.3 (OC), Q5.5
Other:
- note removed: "On va regrouper les labels usb- et out- sur GND pour qu'ils soient regroupé sur le schéma"
- note removed: "j'ai l'impression que les signaux 2 et 5 du 8205 sont inversés"
- note removed: "rajouter connecteur USB C"
- note removed: "rajouter connecteur bloc pile"
- note removed: "regrouper sur un seul label"
Changed lines of the file:
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@@
 	(generator_version "9.0")
 	(paper "A4")
-	(text "On va regrouper les labels usb- et out- sur GND pour qu'ils soient regroupé sur le schéma"
-		(exclude_from_sim no)
-		(at 105.156 138.43 0)
-		(effects
-			(font
-				(size 1.27 1.27)
-				(color 255 0 0 1)
-			)
-		)
-	)
 	(text "Alimenation écran\n"
 		(exclude_from_sim no)
@@
 		)
 	)
-	(text "regrouper sur un seul label"
-		(exclude_from_sim no)
-		(at 197.612 98.552 0)
-		(effects
-			(font
-				(size 1.27 1.27)
-				(color 255 0 0 1)
-			)
-		)
-	)
 	(text "prévoir R16\nau moins 1/4W"
 		(exclude_from_sim no)
@@
 		)
 	)
-	(text "j'ai l'impression que les signaux\n2 et 5 du 8205 sont inversés"
-		(exclude_from_sim no)
-		(at 145.796 132.334 0)
-		(effects
-			(font
-				(size 1.27 1.27)
-				(color 255 0 0 1)
-			)
-		)
-	)
 	(text "Buckboost\n"
 		(exclude_from_sim no)
@@
 		)
 	)
-	(text "rajouter connecteur bloc pile"
-		(exclude_from_sim no)
-		(at 215.138 108.712 0)
-		(effects
-			(font
-				(size 1.27 1.27)
-				(color 255 0 0 1)
-			)
-		)
-	)
-	(text "rajouter connecteur USB C"
-		(exclude_from_sim no)
-		(at 27.686 94.996 0)
-		(effects
-			(font
-				(size 1.27 1.27)
-				(color 255 0 0 1)
-			)
-		)
-	)
 	(text "Bloc régulation de charge\n"
 		(exclude_from_sim no)
@@
 	)
 	(junction
+		(at 27.94 129.54)
+		(diameter 0)
+		(color 0 0 0 0)
+	)
+	(junction
 		(at 82.55 129.54)
 		(diameter 0)
@@
 	)
 	(junction
-		(at 182.88 129.54)
-		(diameter 0)
-		(color 0 0 0 0)
-	)
-	(junction
 		(at 224.79 29.21)
 		(diameter 0)
@@
 	)
 	(junction
-		(at 27.94 129.54)
-		(diameter 0)
-		(color 0 0 0 0)
-	)
-	(junction
 		(at 80.01 129.54)
 		(diameter 0)
@@
 	(wire
 		(pts
-			(xy 25.4 129.54) (xy 27.94 129.54)
-		)
-		(stroke
-			(width 0)
-			(type default)
-		)
-	)
-	(wire
-		(pts
 			(xy 48.26 34.29) (xy 48.26 35.56)
 		)
@@
 	(wire
 		(pts
-			(xy 139.7 127) (xy 139.7 128.27)
-		)
-		(stroke
-			(width 0)
-			(type default)
-		)
-	)
-	(wire
-		(pts
 			(xy 27.94 101.6) (xy 27.94 104.14)
 		)
@@
 	(wire
 		(pts
-			(xy 170.18 116.84) (xy 170.18 128.27)
+			(xy 170.18 116.84) (xy 170.18 121.92)
 		)
 		(stroke
@@
 	(wire
 		(pts
-			(xy 170.18 128.27) (xy 139.7 128.27)
+			(xy 137.16 53.34) (xy 139.7 53.34)
 		)
 		(stroke
@@
 	(wire
 		(pts
-			(xy 137.16 53.34) (xy 139.7 53.34)
+			(xy 170.18 33.02) (xy 176.53 33.02)
 		)
 		(stroke
@@
 	(wire
 		(pts
-			(xy 170.18 33.02) (xy 176.53 33.02)
+			(xy 130.81 127) (xy 139.7 127)
 		)
 		(stroke
@@
 	(wire
 		(pts
+			(xy 27.94 129.54) (xy 27.94 132.08)
+		)
+		(stroke
+			(width 0)
+			(type default)
+		)
+	)
+	(wire
+		(pts
+			(xy 152.4 121.92) (xy 170.18 121.92)
+		)
+		(stroke
+			(width 0)
+			(type default)
+		)
+	)
+	(wire
+		(pts
 			(xy 166.37 116.84) (xy 170.18 116.84)
 		)
@@
 	(wire
 		(pts
-			(xy 129.54 111.76) (xy 129.54 104.14)
+			(xy 130.81 104.14) (xy 130.81 127)
 		)
 		(stroke
@@
 	(wire
 		(pts
-			(xy 182.88 129.54) (xy 186.69 129.54)
-		)
-		(stroke
-			(width 0)
-			(type default)
-		)
-	)
-	(wire
-		(pts
 			(xy 88.9 33.02) (xy 97.79 33.02)
 		)
@@
 	(wire
 		(pts
-			(xy 152.4 121.92) (xy 152.4 111.76)
-		)
-		(stroke
-			(width 0)
-			(type default)
-		)
-	)
-	(wire
-		(pts
 			(xy 146.05 40.64) (xy 146.05 43.18)
 		)
@@
 	(wire
 		(pts
-			(xy 129.54 104.14) (xy 130.81 104.14)
-		)
-		(stroke
-			(width 0)
-			(type default)
-		)
-	)
-	(wire
-		(pts
 			(xy 170.18 109.22) (xy 170.18 116.84)
 		)
@@
 	(wire
 		(pts
-			(xy 152.4 111.76) (xy 129.54 111.76)
-		)
-		(stroke
-			(width 0)
-			(type default)
-		)
-	)
-	(wire
-		(pts
 			(xy 146.05 33.02) (xy 153.67 33.02)
 		)
@@
 		)
 	)
-	(global_label "USB-"
-		(shape input)
-		(at 25.4 129.54 180)
-		(fields_autoplaced yes)
-		(effects
-			(font
-				(size 1.27 1.27)
-			)
-			(justify right)
-		)
-		(property "Intersheetrefs" "${INTERSHEET_REFS}"
-			(at 17.0324 129.54 0)
-			(effects
-				(font
-					(size 1.27 1.27)
-				)
-				(justify right)
-				(hide yes)
-			)
-		)
-	)
 	(global_label "EPD_PWR"
 		(shape input)
@@
 		)
 	)
-	(global_label "OUT-"
-		(shape input)
-		(at 186.69 129.54 0)
-		(fields_autoplaced yes)
-		(effects
-			(font
-				(size 1.27 1.27)
-			)
-			(justify left)
-		)
-		(property "Intersheetrefs" "${INTERSHEET_REFS}"
-			(at 194.8762 129.54 0)
-			(effects
-				(font
-					(size 1.27 1.27)
-				)
-				(justify left)
-				(hide yes)
-			)
-		)
-	)
 	(global_label "CMD_ALIM_SCREEN"
 		(shape input)
@@
 		)
 	)
-	(global_label "OUT+"
-		(shape input)
-		(at 212.09 95.25 270)
-		(fields_autoplaced yes)
-		(effects
-			(font
-				(size 1.27 1.27)
-			)
-			(justify right)
-		)
-		(property "Intersheetrefs" "${INTERSHEET_REFS}"
-			(at 212.09 103.4362 90)
-			(effects
-				(font
-					(size 1.27 1.27)
-				)
-				(justify right)
-				(hide yes)
-			)
-		)
-	)
 	(global_label "VIN"
 		(shape input)
@@
 					(unit 1)
 				)
+			)
+		)
+	)
+	(symbol
+		(lib_id "power:GND")
+		(at 27.94 132.08 0)
+		(unit 1)
+		(exclude_from_sim no)
+		(in_bom yes)
+		(on_board yes)
+		(dnp no)
+		(fields_autoplaced yes)
+		(property "Reference" "#PWR039"
+			(at 27.94 138.43 0)
+			(effects
+				(font
+					(size 1.27 1.27)
+				)
+				(hide yes)
+			)
+		)
+		(property "Value" "GND"
+			(at 27.94 137.16 0)
+			(effects
+				(font
+					(size 1.27 1.27)
+				)
+			)
+		)
+		(property "Footprint" ""
+			(at 27.94 132.08 0)
+			(effects
+				(font
+					(size 1.27 1.27)
+				)
+				(hide yes)
+			)
+		)
+		(property "Datasheet" ""
+			(at 27.94 132.08 0)
+			(effects
+				(font
+					(size 1.27 1.27)
+				)
+				(hide yes)
+			)
+		)
+		(property "Description" "Power symbol creates a global label with name \"GND\" , ground"
+			(at 27.94 132.08 0)
+			(effects
+				(font
+					(size 1.27 1.27)
+				)
+				(hide yes)
+			)
+		)
+		(pin "1"
+		)
+		(instances
+			(project "Station_Meteo_pcb"
+				(path "/90bd0b60-6e70-43e1-8410-99fb54688c17/46b21e09-ea67-4534-a48d-e2dad69aede0"
+					(reference "#PWR039")
+					(unit 1)
+				)

Commit message: t
Parts:
- removed IC1: DW01S, Composants_Perso:DW01S, symbol DW01S:DW01S
- added U5: DW01A, Package_TO_SOT_SMD:SOT-23-6, symbol Battery_Management:DW01A
Connections:
- net BAT-: now also U5.6 (GND)
- net at C17.1, R16.1: now also U5.5 (VCC)
- net at R17.1: now also U5.2 (CS)
- net at Q5.4: now also U5.1 (OD)
- net at Q5.5: now also U5.3 (OC)
- no-connect marks 2 -> 1

Commit message: schema v1
Parts:
- removed Q2, Q4, Q8: PMOS, symbol Simulation_SPICE:PMOS
- removed Q3, Q6: NMOS, symbol Simulation_SPICE:NMOS
- removed R8, R9: 1M, symbol Device:R
- added Q6, Q8: AO3401A, Package_TO_SOT_SMD:SOT-23, symbol Transistor_FET:AO3401A
- added Q9: AO3400A, Package_TO_SOT_SMD:SOT-23, symbol Transistor_FET:AO3400A
- added R26: 0, symbol Device:R
- added TP24, TP25, TP26: TestPoint, symbol Connector:TestPoint
- D4: value LED -> KT-0603W; LCSC (none) -> C2290
- D5: value LED -> KT-0603R; LCSC (none) -> C2286
- R13: value 1k -> 480
- R14: value 1k -> 160
Connections:
- net +3V3: now also R26.2; no longer C15.1, R10.1, R11.1, U4.6 (VOUT)
- net CMD_ALIM_BATTERY: now also Q9.1 (G)
- net GND: now also Q9.2 (S)
- net USB+: no longer C16.1, C29.2, D4.2 (A), D5.2 (A), D6.2 (A), R6.2, U3.4 (V_{CC}), U3.8 (CE)
- net at R23.1: now also Q6.3 (D)
- net at R22.2: now also Q6.1 (G), Q9.3 (D)
- net at Q5.4: now also U5.3 (OC); no longer U5.1 (OD)
- net at Q5.5: now also U5.1 (OD); no longer U5.3 (OC)
- net BAT+ renamed +BATT
- net +BATT: now also Q6.2 (S), Q8.3 (D), TP26.1
- net BAT- renamed GNDA
- net VIN renamed VCC
- net VCC: now also Q8.2 (S), TP24.1
- new net: C15.1, R10.1, R11.1, R26.1, U4.6 (VOUT)
- new net VBUS: C16.1, C29.2, D4.2 (A), D5.2 (A), D6.2 (A), Q8.1 (G), R6.2, TP25.1, U3.4 (V_{CC}), U3.8 (CE)
Other:
- note added: "0603"
- note added: "BAT-"
- note removed: "Alimenation écran"
- note removed: "prévoir R16 au moins 1/4W"
- note removed: "vérif valeur R en fonction de la ref de LED choisi"
- moved on the sheet: D4, D5, R23, R24

Commit message: Connecteurs + sourcing
Parts:
- removed R26: 0, symbol Device:R
- added J10: Conn_01x02_Pin, Connector_PinHeader_2.54mm:PinHeader_1x02_P2.54mm_Vertical_SMD_Pin1Right, symbol Connector:Conn_01x02_Pin
- added R35: 9,1k, Resistor_SMD:R_0603_1608Metric, symbol Device:R
- C13, C15: footprint (none) -> Capacitor_SMD:C_0603_1608Metric; LCSC (none) -> C1523
- C16, C17: footprint (none) -> Capacitor_SMD:C_0402_1005Metric; LCSC (none) -> C1525
- C18, C29: footprint (none) -> Capacitor_SMD:C_0603_1608Metric; LCSC (none) -> C19702
- D4, D5: footprint (none) -> LED_SMD:LED_0603_1608Metric
- R10, R11, R13, R14, R15, R16, R17, R21, R22, R23, R24, R6: footprint (none) -> Resistor_SMD:R_0603_1608Metric
- R12: value 91k -> 82k; footprint (none) -> Resistor_SMD:R_0603_1608Metric
- TP24, TP25, TP26: footprint (none) -> TestPoint:TestPoint_Pad_D1.5mm
Connections:
- net +3V3: now also J10.1 (Pin_1)
- net GND: now also R35.2; no longer R12.2
- net at C15.1, R10.1, R11.1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: now also J10.2 (Pin_2)
- new net: R12.2, R35.1

Commit message: t
Parts:
- removed J10: Conn_01x02_Pin, Connector_PinHeader_2.54mm:PinHeader_1x02_P2.54mm_Vertical_SMD_Pin1Right, symbol Connector:Conn_01x02_Pin
- added J4: DZ254S-11-02-48, Connector_PinHeader_2.54mm:PinHeader_1x02_P2.54mm_Vertical_SMD_Pin1Right, symbol Connector:Conn_01x02_Pin
- added J8: Conn_01x02_Pin, Connector_PinHeader_2.54mm:PinHeader_1x02_P2.54mm_Vertical_SMD_Pin1Left, symbol Connector:Conn_01x02_Pin
Connections:
- net +3V3: now also J4.1 (Pin_1)
- net VCC: now also J8.1 (Pin_1); no longer D6.1 (K), Q8.2 (S)
- net at C15.1, R10.1, R11.1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: now also J4.2 (Pin_2)
- new net: D6.1 (K), J8.2 (Pin_2), Q8.2 (S)
Other:
- moved on the sheet: C16, C17, C18, C29, D4, D5, D6, Q5, Q8, R13, R14, R15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

Commit message: t
Parts:
- L2: footprint (none) -> Composants_Perso:SPM4030T-R47M-HZ
Changed lines of the file:
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@@
 			)
 		)
-		(property "Footprint" ""
+		(property "Footprint" "Composants_Perso:SPM4030T-R47M-HZ"
 			(at 99.06 50.8 0)
 			(effects

Commit message: t
Parts:
- D6: value 1N5817 -> 1N5817W; footprint Diode_THT:D_DO-41_SOD81_P10.16mm_Horizontal -> Diode_SMD:D_SOD-123; LCSC (none) -> C5185908
- J8: value Conn_01x02_Pin -> DZ254S-11-02-48; LCSC (none) -> C5160785
- L2: LCSC (none) -> C531455
- Q5: LCSC (none) -> C2830320
- Q6, Q8: LCSC (none) -> C15127
- Q9: LCSC (none) -> C20917
- R10, R6: LCSC (none) -> C25803
- R11: LCSC (none) -> C23192
- R12: LCSC (none) -> C23254
- R13: value 480 -> 470; LCSC (none) -> C23179
- R14: value 160 -> 150; LCSC (none) -> C22808
- R15: LCSC (none) -> C22765
- R16: LCSC (none) -> C22775
- R17: LCSC (none) -> C21190
- R21, R22: LCSC (none) -> C22935
- R23: LCSC (none) -> C25804
- R24: value 33K -> 33k; LCSC (none) -> C4216
- R35: value 9,1k -> 9k1; LCSC (none) -> C23260
- TP24, TP25, TP26: now left out of the parts list
- U3: LCSC (none) -> C16581
- U4: LCSC (none) -> C2845237
Other:
- note removed: "0603"
- moved on the sheet: D6

Commit message: Placement + routage V2
Parts:
- renumbered TP26 to BAT1, TP24 to VCC1
Changed lines of the file:
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@@
 		(on_board yes)
 		(dnp no)
-		(property "Reference" "TP24"
+		(property "Reference" "VCC1"
 			(at 95.758 27.432 0)
 			(effects
@@
 			(project "Station_Meteo_pcb"
 				(path "/90bd0b60-6e70-43e1-8410-99fb54688c17/46b21e09-ea67-4534-a48d-e2dad69aede0"
-					(reference "TP24")
+					(reference "VCC1")
 					(unit 1)
 				)
@@
 		(on_board yes)
 		(dnp no)
-		(property "Reference" "TP26"
+		(property "Reference" "BAT1"
 			(at 119.888 87.122 0)
 			(effects
@@
 			(project "Station_Meteo_pcb"
 				(path "/90bd0b60-6e70-43e1-8410-99fb54688c17/46b21e09-ea67-4534-a48d-e2dad69aede0"
-					(reference "TP26")
+					(reference "BAT1")
 					(unit 1)
 				)
