File: Alimentation.kicad_sch (KiCad schematic)
At the start: 36 parts, among them J4 DZ254S-11-02-48, J8 DZ254S-11-02-48, Q5 FS8205A, Q6 AO3401A, Q8 AO3401A, Q9 AO3400A, U3 TP4056-42-ESOP8, U4 TPS63802DLAR, U5 DW01A

Commit message: t
Parts:
- added 3V3, 3V3_1: TestPoint, TestPoint:TestPoint_Pad_D1.5mm, symbol Connector:TestPoint
Connections:
- net +3V3: now also 3V3.1, 3V3_1.1
- net at R14.1: now also U3.7 (~{CHRG}); no longer U3.6 (~{STDBY})
- net at R13.1: now also U3.6 (~{STDBY}); no longer U3.7 (~{CHRG})
Other:
- moved on the sheet: R13, R14

Commit message: modif pour commande
Parts:
- C13, C15: LCSC C1523 -> C59461
- J4: footprint Connector_PinHeader_2.54mm:PinHeader_1x02_P2.54mm_Vertical_SMD_Pin1Right -> Connector_PinHeader_2.54mm:PinHeader_1x02_P2.54mm_Vertical_SMD_Pin1Left
Changed lines of the file:
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@@
 			)
 		)
-		(property "LCSC" "C1523"
+		(property "LCSC" "C59461"
 			(at 97.79 35.56 0)
 			(effects
@@
 			)
 		)
-		(property "Footprint" "Connector_PinHeader_2.54mm:PinHeader_1x02_P2.54mm_Vertical_SMD_Pin1Right"
+		(property "Footprint" "Connector_PinHeader_2.54mm:PinHeader_1x02_P2.54mm_Vertical_SMD_Pin1Left"
 			(at 180.34 27.94 0)
 			(effects
@@
 			)
 		)
-		(property "LCSC" "C1523"
+		(property "LCSC" "C59461"
 			(at 170.18 35.56 0)
 			(effects

Commit message: last p
Parts:
- Q5: value FS8205A -> FH8205A; LCSC C2830320 -> C2929075; MP FS8205A -> FH8205A
Changed lines of the file:
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@@
 			)
 		)
-		(property "Value" "FS8205A"
+		(property "Value" "FH8205A"
 			(at 156.5911 119.38 90)
 			(effects
@@
 			)
 		)
-		(property "MP" "FS8205A"
+		(property "MP" "FH8205A"
 			(at 154.94 124.46 0)
 			(effects
@@
 			)
 		)
-		(property "LCSC" "C2830320"
+		(property "LCSC" "C2929075"
 			(at 154.94 124.46 90)
 			(effects
