File: MCU.kicad_sch (KiCad schematic)
At the start: 20 parts, among them U2 STM32L476RGTx, Y2 Crystal

Commit message: schema v1
Parts:
- added R27, R30, R31, R32, R33, R34: 0, symbol Device:R
- added TP10, TP11, TP12, TP13, TP14, TP15, TP16, TP17, TP18, TP19, TP20, TP21, TP22, TP23, TP6, TP7, TP8, TP9: TestPoint, symbol Connector:TestPoint
Connections:
- net +3.3V: now also R34.2, TP18.1, TP19.1, TP20.1; no longer C20.1, C21.1, C22.1, C23.1, C30.1, U2.1 (VBAT), U2.19 (VDD), U2.32 (VDD), U2.64 (VDD)
- net CMD_ALIM_BATTERY: now also R30.2; no longer U2.9 (PC1)
- net CMD_ALIM_SCREEN: now also R31.1; no longer U2.8 (PC0)
- net EPD_BUSY: now also TP10.1
- net EPD_CS: now also TP9.1
- net EPD_DC: now also TP11.1
- net EPD_DIN: now also TP6.1
- net EPD_PWR: now also TP7.1
- net EPD_RST: now also TP12.1
- net EPD_SCK: now also TP8.1
- net GND: now also TP21.1, TP22.1, TP23.1
- net MEASURE_BATTERY: now also R27.2; no longer U2.11 (PC3)
- net SCL: now also R33.2; no longer U2.61 (PB8)
- net SDA: now also R32.1; no longer U2.62 (PB9)
- new net: R32.2, TP13.1, U2.62 (PB9)
- new net: R30.1, TP16.1, U2.9 (PC1)
- new net: C20.1, C21.1, C22.1, C23.1, C30.1, R34.1, U2.1 (VBAT), U2.19 (VDD), U2.32 (VDD), U2.64 (VDD)
- new net: R27.1, TP15.1, U2.11 (PC3)
- new net: R33.1, TP14.1, U2.61 (PB8)
- new net: R31.2, TP17.1, U2.8 (PC0)

Commit message: Connecteurs + sourcing
Parts:
- removed R27, R30, R31, R32, R33, R34: 0, symbol Device:R
- added J4, J6, J7: Conn_01x02_Pin, Connector_PinHeader_2.54mm:PinHeader_1x02_P2.54mm_Vertical_SMD_Pin1Right, symbol Connector:Conn_01x02_Pin
- added J5, J8, J9: Conn_01x02_Pin, Connector_PinHeader_2.54mm:PinHeader_1x02_P2.54mm_Vertical_SMD_Pin1Left, symbol Connector:Conn_01x02_Pin
- C19: footprint (none) -> Capacitor_SMD:C_0402_1005Metric
- C20: footprint (none) -> Capacitor_SMD:C_0805_2012Metric
- C21, C22, C23, C30, C5: footprint (none) -> Capacitor_SMD:C_0402_1005Metric; LCSC (none) -> C1525
- C24, C28: footprint (none) -> Capacitor_SMD:C_0603_1608Metric; LCSC (none) -> C15849
- C25: footprint (none) -> Capacitor_SMD:C_0603_1608Metric; LCSC (none) -> C57112
- C26, C27: footprint (none) -> Capacitor_SMD:C_0402_1005Metric; LCSC (none) -> C1547
- R5: footprint (none) -> Resistor_SMD:R_0603_1608Metric
- TP1, TP10, TP11, TP12, TP13, TP14, TP15, TP16, TP17, TP18, TP19, TP2, TP20, TP21, TP22, TP23, TP3, TP4, TP5, TP6, TP7, TP8, TP9: footprint (none) -> TestPoint:TestPoint_Pad_D1.5mm
- Y2: footprint (none) -> Crystal:Crystal_SMD_3215-2Pin_3.2x1.5mm
Connections:
- net CMD_ALIM_BATTERY: now also J7.1 (Pin_1)
- net CMD_ALIM_SCREEN: now also J8.2 (Pin_2)
- net MEASURE_BATTERY: now also J6.1 (Pin_1)
- net SCL: now also J5.1 (Pin_1)
- net SDA: now also J4.2 (Pin_2)
- net at TP13.1, U2.62 (PB9): now also J4.1 (Pin_1)
- net at TP16.1, U2.9 (PC1): now also J7.2 (Pin_2)
- net at C20.1, C21.1, C22.1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: now also J9.1 (Pin_1)
- net at TP15.1, U2.11 (PC3): now also J6.2 (Pin_2)
- net at TP14.1, U2.61 (PB8): now also J5.2 (Pin_2)
- net at TP17.1, U2.8 (PC0): now also J8.1 (Pin_1)
- net +3.3V renamed +3V3
- net +3V3: now also J9.2 (Pin_2)

Commit message: t
Parts:
- removed J4, J6, J7: Conn_01x02_Pin, Connector_PinHeader_2.54mm:PinHeader_1x02_P2.54mm_Vertical_SMD_Pin1Right, symbol Connector:Conn_01x02_Pin
- removed J5, J8: Conn_01x02_Pin, Connector_PinHeader_2.54mm:PinHeader_1x02_P2.54mm_Vertical_SMD_Pin1Left, symbol Connector:Conn_01x02_Pin
Connections:
- net CMD_ALIM_BATTERY: now also TP16.1, U2.9 (PC1)
- net CMD_ALIM_SCREEN: now also TP17.1, U2.8 (PC0)
- net MEASURE_BATTERY: now also TP15.1, U2.11 (PC3)
- net SCL: now also TP14.1, U2.61 (PB8)
- net SDA: now also TP13.1, U2.62 (PB9)

Commit message: t
Parts:
- removed TP2: TestPoint_Small, TestPoint:TestPoint_Pad_D1.5mm, symbol Connector:TestPoint_Small
- added TP2: TestPoint, TestPoint:TestPoint_Pad_D1.5mm, symbol Connector:TestPoint
- C19: LCSC (none) -> C1525
- C20: value 4.7u -> 4.7u/25V; LCSC (none) -> C1779
- C24, C28: value 1u -> 1u/50
- J9: value Conn_01x02_Pin -> DZ254S-11-02-48; LCSC (none) -> C5160785
- R5: LCSC (none) -> C25804
- TP1, TP10, TP11, TP12, TP13, TP14, TP15, TP16, TP17, TP18, TP19, TP20, TP21, TP22, TP23, TP3, TP4, TP5, TP6, TP7, TP8, TP9: now left out of the parts list
- U2: LCSC (none) -> C74797
- Y2: LCSC (none) -> C2450907
Connections:
- net nRST: now also TP2.1
Other:
- note removed: "ECX-.327-CDX-1293"

Commit message: t
Parts:
- removed TP10, TP11, TP12, TP17, TP6, TP7, TP8, TP9: TestPoint, TestPoint:TestPoint_Pad_D1.5mm, symbol Connector:TestPoint
Connections:
- net CMD_ALIM_SCREEN: no longer names the net of U2.8 (PC0)
- no-connect marks 32 -> 33

Commit message: revue
Connections:
- net +3V3: no longer C24.1, C25.1, C28.1, C5.1, TP18.1, TP19.1, TP20.1, U2.13 (VDDA), U2.48 (VDDUSB)
- net 3v3s: now reaches C20.1, C21.1, C22.1, C23.1, C30.1, J9.1 (Pin_1), U2.1 (VBAT), U2.19 (VDD), U2.32 (VDD), U2.64 (VDD)
- net 3v3s: now also C24.1, C25.1, C28.1, C5.1, TP18.1, TP19.1, TP20.1, U2.13 (VDDA), U2.48 (VDDUSB)
Changed lines of the file:
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@@
 	)
 	(junction
+		(at 81.28 124.46)
+		(diameter 0)
+		(color 0 0 0 0)
+	)
+	(junction
+		(at 139.7 124.46)
+		(diameter 0)
+		(color 0 0 0 0)
+	)
+	(junction
 		(at 185.42 46.99)
 		(diameter 0)
@@
 	)
 	(junction
+		(at 137.16 124.46)
+		(diameter 0)
+		(color 0 0 0 0)
+	)
+	(junction
 		(at 83.82 120.65)
 		(diameter 0)
@@
 	)
 	(junction
-		(at 72.39 120.65)
+		(at 105.41 124.46)
 		(diameter 0)
 		(color 0 0 0 0)
 	)
 	(junction
-		(at 195.58 124.46)
+		(at 72.39 120.65)
 		(diameter 0)
 		(color 0 0 0 0)
 	)
 	(junction
-		(at 166.37 87.63)
+		(at 195.58 124.46)
 		(diameter 0)
 		(color 0 0 0 0)
 	)
 	(junction
-		(at 72.39 132.08)
+		(at 166.37 87.63)
 		(diameter 0)
 		(color 0 0 0 0)
 	)
 	(junction
-		(at 105.41 124.46)
+		(at 72.39 132.08)
 		(diameter 0)
 		(color 0 0 0 0)
@@
 	(wire
 		(pts
+			(xy 137.16 124.46) (xy 139.7 124.46)
+		)
+		(stroke
+			(width 0)
+			(type default)
+		)
+	)
+	(wire
+		(pts
 			(xy 95.25 120.65) (xy 134.62 120.65)
 		)
@@
 	(wire
 		(pts
+			(xy 81.28 124.46) (xy 105.41 124.46)
+		)
+		(stroke
+			(width 0)
+			(type default)
+		)
+	)
+	(wire
+		(pts
 			(xy 72.39 129.54) (xy 72.39 132.08)
 		)
@@
 	(wire
 		(pts
-			(xy 66.04 124.46) (xy 72.39 124.46)
-		)
-		(stroke
-			(width 0)
-			(type default)
-		)
-	)
-	(wire
-		(pts
 			(xy 191.77 124.46) (xy 195.58 124.46)
 		)
@@
 		)
 	)
+	(global_label "3v3s"
+		(shape input)
+		(at 130.81 124.46 270)
+		(fields_autoplaced yes)
+		(effects
+			(font
+				(size 1.27 1.27)
+			)
+			(justify right)
+		)
+		(property "Intersheetrefs" "${INTERSHEET_REFS}"
+			(at 130.81 131.8599 90)
+			(effects
+				(font
+					(size 1.27 1.27)
+				)
+				(justify right)
+				(hide yes)
+			)
+		)
+	)
 	(global_label "MEASURE_BATTERY"
 		(shape input)
@@
 	(symbol
 		(lib_id "power:+3.3V")
-		(at 66.04 124.46 90)
-		(unit 1)
-		(exclude_from_sim no)
-		(in_bom yes)
-		(on_board yes)
-		(dnp no)
-		(property "Reference" "#PWR013"
-			(at 69.85 124.46 0)
-			(effects
-				(font
-					(size 1.27 1.27)
-				)
-				(hide yes)
-			)
-		)
-		(property "Value" "+3V3"
-			(at 62.23 124.4601 90)
-			(effects
-				(font
-					(size 1.27 1.27)
-				)
-				(justify left)
-			)
-		)
-		(property "Footprint" ""
-			(at 66.04 124.46 0)
-			(effects
-				(font
-					(size 1.27 1.27)
-				)
-				(hide yes)
-			)
-		)
-		(property "Datasheet" ""
-			(at 66.04 124.46 0)
-			(effects
-				(font
-					(size 1.27 1.27)
-				)
-				(hide yes)
-			)
-		)
-		(property "Description" "Power symbol creates a global label with name \"+3.3V\""
-			(at 66.04 124.46 0)
-			(effects
-				(font
-					(size 1.27 1.27)
-				)
-				(hide yes)
-			)
-		)
-		(pin "1"
-		)
-		(instances
-			(project "Station_Meteo_pcb"
-				(path "/90bd0b60-6e70-43e1-8410-99fb54688c17/9ce3ae06-c5cc-4000-b6d8-5ae3d540ff9d"
-					(reference "#PWR013")
-					(unit 1)
-				)
-			)
-		)
-	)
-	(symbol
-		(lib_id "power:+3.3V")
 		(at 209.55 124.46 270)
 		(unit 1)
@@
 					(unit 1)
 				)
-			)
-		)
-	)
-	(symbol
-		(lib_id "power:+3.3V")
-		(at 105.41 124.46 90)
-		(unit 1)
-		(exclude_from_sim no)
-		(in_bom yes)
-		(on_board yes)
-		(dnp no)
-		(property "Reference" "#PWR012"
-			(at 109.22 124.46 0)
-			(effects
-				(font
-					(size 1.27 1.27)
-				)
-				(hide yes)
-			)
-		)
-		(property "Value" "+3V3"
-			(at 101.6 124.4601 90)
-			(effects
-				(font
-					(size 1.27 1.27)
-				)
-				(justify left)
-			)
-		)
-		(property "Footprint" ""
-			(at 105.41 124.46 0)
-			(effects
-				(font
-					(size 1.27 1.27)
-				)
-				(hide yes)
-			)
-		)
-		(property "Datasheet" ""
-			(at 105.41 124.46 0)
-			(effects
-				(font
-					(size 1.27 1.27)
-				)
-				(hide yes)
-			)
-		)
-		(property "Description" "Power symbol creates a global label with name \"+3.3V\""
-			(at 105.41 124.46 0)
-			(effects
-				(font
-					(size 1.27 1.27)
-				)
-				(hide yes)
-			)
-		)
-		(pin "1"
-		)
-		(instances
-			(project "Station_Meteo_pcb"
-				(path "/90bd0b60-6e70-43e1-8410-99fb54688c17/9ce3ae06-c5cc-4000-b6d8-5ae3d540ff9d"
-					(reference "#PWR012")
-					(unit 1)
-				)

Commit message: Placement + routage V2
Parts:
- renumbered TP1 to BOOT1, TP16 to CMD_BAT1, TP3 to DEBUG1, TP4 to DEBUG2, TP5 to DEBUG3, TP23 to GND1, TP21 to GND2, TP22 to GND3, TP15 to MEAS_BAT1, TP14 to SCL1, TP13 to SDA1, TP2 to nRST1
Connections:
- net 3v3s: no longer names the net of C20.1, C21.1, C22.1, C23.1, C24.1, C25.1, C28.1, C30.1, C5.1, J9.1 (Pin_1), TP18.1, TP19.1, TP20.1, U2.1 (VBAT), U2.13 (VDDA), U2.19 (VDD), U2.32 (VDD), U2.48 (VDDUSB), U2.64 (VDD)
Changed lines of the file:
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@@
 		)
 	)
-	(global_label "3v3s"
-		(shape input)
-		(at 130.81 124.46 270)
-		(fields_autoplaced yes)
-		(effects
-			(font
-				(size 1.27 1.27)
-			)
-			(justify right)
-		)
-		(property "Intersheetrefs" "${INTERSHEET_REFS}"
-			(at 130.81 131.8599 90)
-			(effects
-				(font
-					(size 1.27 1.27)
-				)
-				(justify right)
-				(hide yes)
-			)
-		)
-	)
 	(global_label "MEASURE_BATTERY"
 		(shape input)
@@
 		(on_board yes)
 		(dnp no)
-		(property "Reference" "TP13"
+		(property "Reference" "SDA1"
 			(at 116.586 41.148 0)
 			(effects
@@
 			(project "Station_Meteo_pcb"
 				(path "/90bd0b60-6e70-43e1-8410-99fb54688c17/9ce3ae06-c5cc-4000-b6d8-5ae3d540ff9d"
-					(reference "TP13")
+					(reference "SDA1")
 					(unit 1)
 				)
@@
 		(dnp no)
 		(fields_autoplaced yes)
-		(property "Reference" "TP2"
+		(property "Reference" "nRST1"
 			(at 170.18 110.4899 90)
 			(effects
@@
 			(project "Station_Meteo_pcb"
 				(path "/90bd0b60-6e70-43e1-8410-99fb54688c17/9ce3ae06-c5cc-4000-b6d8-5ae3d540ff9d"
-					(reference "TP2")
+					(reference "nRST1")
 					(unit 1)
 				)
@@
 		(on_board yes)
 		(dnp no)
-		(property "Reference" "TP4"
+		(property "Reference" "DEBUG2"
 			(at 115.316 61.468 0)
 			(effects
@@
 			(project "Station_Meteo_pcb"
 				(path "/90bd0b60-6e70-43e1-8410-99fb54688c17/9ce3ae06-c5cc-4000-b6d8-5ae3d540ff9d"
-					(reference "TP4")
+					(reference "DEBUG2")
 					(unit 1)
 				)
@@
 		(on_board yes)
 		(dnp no)
-		(property "Reference" "TP3"
+		(property "Reference" "DEBUG1"
 			(at 115.316 23.368 0)
 			(effects
@@
 			(project "Station_Meteo_pcb"
 				(path "/90bd0b60-6e70-43e1-8410-99fb54688c17/9ce3ae06-c5cc-4000-b6d8-5ae3d540ff9d"
-					(reference "TP3")
+					(reference "DEBUG1")
 					(unit 1)
 				)
@@
 		(on_board yes)
 		(dnp no)
-		(property "Reference" "TP22"
+		(property "Reference" "GND3"
 			(at 131.318 14.732 0)
 			(effects
@@
 			(project "Station_Meteo_pcb"
 				(path "/90bd0b60-6e70-43e1-8410-99fb54688c17/9ce3ae06-c5cc-4000-b6d8-5ae3d540ff9d"
-					(reference "TP22")
+					(reference "GND3")
 					(unit 1)
 				)
@@
 		(on_board yes)
 		(dnp no)
-		(property "Reference" "TP16"
+		(property "Reference" "CMD_BAT1"
 			(at 161.036 86.106 0)
 			(effects
@@
 			(project "Station_Meteo_pcb"
 				(path "/90bd0b60-6e70-43e1-8410-99fb54688c17/9ce3ae06-c5cc-4000-b6d8-5ae3d540ff9d"
-					(reference "TP16")
+					(reference "CMD_BAT1")
 					(unit 1)
 				)
@@
 		(on_board yes)
 		(dnp no)
-		(property "Reference" "TP15"
+		(property "Reference" "MEAS_BAT1"
 			(at 162.306 76.708 0)
 			(effects
@@
 			(project "Station_Meteo_pcb"
 				(path "/90bd0b60-6e70-43e1-8410-99fb54688c17/9ce3ae06-c5cc-4000-b6d8-5ae3d540ff9d"
-					(reference "TP15")
+					(reference "MEAS_BAT1")
 					(unit 1)
 				)
@@
 		(on_board yes)
 		(dnp no)
-		(property "Reference" "TP14"
+		(property "Reference" "SCL1"
 			(at 119.634 55.372 0)
 			(effects
@@
 			(project "Station_Meteo_pcb"
 				(path "/90bd0b60-6e70-43e1-8410-99fb54688c17/9ce3ae06-c5cc-4000-b6d8-5ae3d540ff9d"
-					(reference "TP14")
+					(reference "SCL1")
 					(unit 1)
 				)
@@
 		(on_board yes)
 		(dnp no)
-		(property "Reference" "TP23"
+		(property "Reference" "GND1"
 			(at 118.618 14.732 0)
 			(effects
@@
 			(project "Station_Meteo_pcb"
 				(path "/90bd0b60-6e70-43e1-8410-99fb54688c17/9ce3ae06-c5cc-4000-b6d8-5ae3d540ff9d"
-					(reference "TP23")
+					(reference "GND1")
 					(unit 1)
 				)
@@
 		(dnp no)
 		(fields_autoplaced yes)
-		(property "Reference" "TP1"
-			(at 177.8 106.6799 90)
+		(property "Reference" "BOOT1"
+			(at 177.8 107.9499 90)
 			(effects
 				(font
@@
 			(project ""
 				(path "/90bd0b60-6e70-43e1-8410-99fb54688c17/9ce3ae06-c5cc-4000-b6d8-5ae3d540ff9d"
-					(reference "TP1")
+					(reference "BOOT1")
 					(unit 1)
 				)
@@
 		(on_board yes)
 		(dnp no)
-		(property "Reference" "TP5"
+		(property "Reference" "DEBUG3"
 			(at 169.164 64.262 0)
 			(effects
@@
 			(project "Station_Meteo_pcb"
 				(path "/90bd0b60-6e70-43e1-8410-99fb54688c17/9ce3ae06-c5cc-4000-b6d8-5ae3d540ff9d"
-					(reference "TP5")
+					(reference "DEBUG3")
 					(unit 1)
 				)
@@
 		(on_board yes)
 		(dnp no)
-		(property "Reference" "TP21"
+		(property "Reference" "GND2"
 			(at 124.968 14.732 0)
 			(effects
@@
 			(project "Station_Meteo_pcb"
 				(path "/90bd0b60-6e70-43e1-8410-99fb54688c17/9ce3ae06-c5cc-4000-b6d8-5ae3d540ff9d"
-					(reference "TP21")
+					(reference "GND2")
 					(unit 1)
 				)

Commit message: t
Parts:
- removed DEBUG3, TP18, TP19: TestPoint, TestPoint:TestPoint_Pad_D1.5mm, symbol Connector:TestPoint
Connections:
- net DEBUG3: no longer names the net of U2.38 (PC7)
- no-connect marks 33 -> 34
