File: MCU.kicad_sch (KiCad schematic)
At the start: 28 parts, among them J9 DZ254S-11-02-48, U2 STM32L476RGTx, Y2 Crystal

Commit message: Placement + routage V3
Parts:
- renumbered TP20 to VDD1
Changed lines of the file:
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@@
 	)
 	(junction
-		(at 139.7 21.59)
-		(diameter 0)
-		(color 0 0 0 0)
-	)
-	(junction
 		(at 118.11 46.99)
 		(diameter 0)
@@
 	)
 	(junction
-		(at 165.1 113.03)
+		(at 139.7 21.59)
 		(diameter 0)
 		(color 0 0 0 0)
 	)
 	(junction
-		(at 118.11 49.53)
+		(at 165.1 113.03)
 		(diameter 0)
 		(color 0 0 0 0)
 	)
 	(junction
-		(at 114.3 124.46)
+		(at 118.11 49.53)
 		(diameter 0)
 		(color 0 0 0 0)
 	)
 	(junction
-		(at 140.97 21.59)
+		(at 114.3 124.46)
 		(diameter 0)
 		(color 0 0 0 0)
@@
 	(wire
 		(pts
+			(xy 142.24 21.59) (xy 142.24 24.13)
+		)
+		(stroke
+			(width 0)
+			(type default)
+		)
+	)
+	(wire
+		(pts
 			(xy 113.03 105.41) (xy 124.46 105.41)
 		)
@@
 	(wire
 		(pts
-			(xy 140.97 21.59) (xy 142.24 21.59)
-		)
-		(stroke
-			(width 0)
-			(type default)
-		)
-	)
-	(wire
-		(pts
 			(xy 203.2 124.46) (xy 209.55 124.46)
 		)
@@
 	(wire
 		(pts
+			(xy 139.7 20.32) (xy 139.7 21.59)
+		)
+		(stroke
+			(width 0)
+			(type default)
+		)
+	)
+	(wire
+		(pts
 			(xy 142.24 124.46) (xy 139.7 124.46)
 		)
@@
 	(wire
 		(pts
-			(xy 140.97 20.32) (xy 140.97 21.59)
+			(xy 113.03 97.79) (xy 124.46 97.79)
 		)
 		(stroke
@@
 	(wire
 		(pts
-			(xy 113.03 97.79) (xy 124.46 97.79)
+			(xy 139.7 21.59) (xy 142.24 21.59)
 		)
 		(stroke
@@
 	(wire
 		(pts
-			(xy 142.24 21.59) (xy 142.24 24.13)
-		)
-		(stroke
-			(width 0)
-			(type default)
-		)
-	)
-	(wire
-		(pts
 			(xy 144.78 124.46) (xy 147.32 124.46)
 		)
@@
 	(wire
 		(pts
-			(xy 139.7 21.59) (xy 140.97 21.59)
-		)
-		(stroke
-			(width 0)
-			(type default)
-		)
-	)
-	(wire
-		(pts
 			(xy 114.3 129.54) (xy 114.3 132.08)
 		)
@@
 		(on_board yes)
 		(dnp no)
-		(property "Reference" "TP20"
+		(property "Reference" "VDD1"
 			(at 96.774 118.11 0)
 			(effects
@@
 			(project "Station_Meteo_pcb"
 				(path "/90bd0b60-6e70-43e1-8410-99fb54688c17/9ce3ae06-c5cc-4000-b6d8-5ae3d540ff9d"
-					(reference "TP20")
+					(reference "VDD1")
 					(unit 1)
 				)
@@
 	(symbol
 		(lib_id "power:GND")
-		(at 140.97 20.32 180)
+		(at 139.7 20.32 180)
 		(unit 1)
 		(exclude_from_sim no)
@@
 		(fields_autoplaced yes)
 		(property "Reference" "#PWR024"
-			(at 140.97 13.97 0)
+			(at 139.7 13.97 0)
 			(effects
 				(font
@@
 		)
 		(property "Value" "GND"
-			(at 140.97 15.24 0)
+			(at 139.7 15.24 0)
 			(effects
 				(font
@@
 		)
 		(property "Footprint" ""
-			(at 140.97 20.32 0)
+			(at 139.7 20.32 0)
 			(effects
 				(font
@@
 		)
 		(property "Datasheet" ""
-			(at 140.97 20.32 0)
+			(at 139.7 20.32 0)
 			(effects
 				(font
@@
 		)
 		(property "Description" "Power symbol creates a global label with name \"GND\" , ground"
-			(at 140.97 20.32 0)
+			(at 139.7 20.32 0)
 			(effects
 				(font

Commit message: modif pour commande
Parts:
- C24, C28: value 1u/50 -> 1u/50V
Changed lines of the file:
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@@
 			)
 		)
-		(property "Value" "1u/50"
+		(property "Value" "1u/50V"
 			(at 83.82 130.048 0)
 			(effects
@@
 			)
 		)
-		(property "Value" "1u/50"
+		(property "Value" "1u/50V"
 			(at 116.84 130.048 0)
 			(effects
