File: Station_Meteo_pcb.kicad_pcb (KiCad board)
At the start: 2 copper layers, 107 x 64 mm, 124 parts, among them J1 ZX-FPC-FWSX0.5PH224, J10 DZ254S-11-02-48, J11 DZ254S-11-02-48, J2 UC18-0B06F68011, J3 BH127VS-14P-H49, J4 DZ254S-11-02-48, J5 DZ254S-11-02-48, J6 DZ254S-11-02-48, J8 DZ254S-11-02-48, J9 DZ254S-11-02-48, Q1 AO3400A, Q2 AO3400A, Q3 AO3401A, Q5 FS8205A, Q6 AO3401A, Q7 AO3401A, Q8 AO3401A, Q9 AO3400A, U1 BME280, U2 STM32L476RGTx, U3 TP4056-42-ESOP8, U4 TPS63802DLAR, U5 DW01A, Y2 Crystal

Commit message: TEST POINT
Parts:
- moved TP14 146.6 mm to (117.2, 57.0)
- moved TP22 140.4 mm to (130.8, 62.5)
- moved TP13 138.5 mm to (121.2, 57.8)
- moved TP29 133.0 mm to (127.4, 85.5)
- moved TP28 131.3 mm to (130.8, 85.3)
- moved TP27 126.9 mm to (134.9, 80.2)
- moved TP18 119.7 mm to (147.9, 56.8)
- moved TP31 119.2 mm to (136.0, 75.8)
- moved TP19 118.0 mm to (155.7, 84.2)
- moved TP30 117.7 mm to (137.2, 70.9)
- moved TP1 113.3 mm to (145.3, 65.0)
- moved TP16 109.0 mm to (157.3, 74.1)
- moved TP15 108.1 mm to (158.7, 72.4)
- moved TP5 104.0 mm to (155.4, 49.0)
- moved TP32 103.6 mm to (184.9, 92.5)
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Routing:
- net Net-(D3-K): track 12.9 -> 15.8 mm
- net Net-(D2-K): track 7.27 -> 8.73 mm
- net Net-(D1-A): track 18.6 -> 17.5 mm
- net RESE: track 12.7 -> 13.5 mm
- net GDR: track 10.9 -> 11.6 mm

Commit message: Placement + routage V2
Parts:
- moved TP19 16.1 mm to (163.0, 69.8)
- moved CMD_BAT1 0.61 mm to (157.4, 74.7)
- moved R21 0.51 mm to (157.6, 77.5)
- moved BOOT1 0.23 mm to (145.5, 64.9)
- renumbered TP27 to ALIM_S1, TP32 to BAT+1, TP26 to BAT1, TP1 to BOOT1, TP16 to CMD_BAT1, TP3 to DEBUG1, TP4 to DEBUG2, TP5 to DEBUG3, TP23 to GND1, TP21 to GND2, TP22 to GND3, TP15 to MEAS_BAT1, TP28 to RESE1, TP14 to SCL1, TP13 to SDA1, TP33 to VBUS1, TP24 to VCC1, TP2 to nRST1
Connections:
- net 3v3s renamed Net-(J9-Pin_1)
Routing:
- net CMD_ALIM_BATTERY: track 11.9 -> 12.6 mm
- net GND: track 17.0 -> 16.3 mm, vias 10 -> 11

Commit message: t
Parts:
- removed DEBUG3, TP18, TP19: TestPoint, TestPoint:TestPoint_Pad_D1.5mm
- added 3V3: TestPoint, TestPoint:TestPoint_Pad_D1.5mm, F.Cu at (153.4, 84.2)
- added 3V3_1: TestPoint, TestPoint:TestPoint_Pad_D1.5mm, F.Cu at (178.2, 69.8)
- moved D5 61.5 mm to (205.2, 57.9), turned to 90 degrees
- moved D4 60.3 mm to (205.2, 52.8), turned to 90 degrees
- moved R13 50.0 mm to (218.7, 60.7)
- moved R14 50.0 mm to (218.7, 63.2)
- moved DEBUG1 6.19 mm to (162.3, 54.1)
- moved R5 4.62 mm to (145.7, 65.5), turned to 90 degrees
- moved BOOT1 2.75 mm to (142.9, 65.8)
- moved C12 0.73 mm to (129.4, 81.6)
- renumbered TP29 to GDR1
Connections:
- R13 pad 1: Net-(U3-~{CHRG}) -> Net-(U3-~{STDBY})
- R14 pad 1: Net-(U3-~{STDBY}) -> Net-(U3-~{CHRG})
- U2 pad 38: DEBUG3 -> unconnected-(U2-PC7-Pad38)
Routing:
- net Net-(U2-BOOT0): track 1.92 -> 12.3 mm, vias 0 -> 2
- net DEBUG1: track 0.00 -> 4.66 mm
- net DEBUG2: track 0.00 -> 2.74 mm
- net GND: track 16.3 -> 18.5 mm, vias 11 -> 18
- net Net-(J1-Pin_5): track 5.35 -> 4.62 mm
- net nRST: vias 2 -> 3
- net SDA: vias 2 -> 3
- net SCL: vias 2 -> 3

Commit message: comit
Parts:
- moved R13 18.5 mm to (202.2, 52.2)
- moved R14 17.3 mm to (202.1, 58.1)
- moved D5 0.60 mm to (205.2, 57.3)
- moved D4 0.25 mm to (205.1, 53.0), turned to -90 degrees
Routing:
- net VBUS: track 35.6 -> 73.8 mm
- net Net-(U3-~{STDBY}): track 0.00 -> 36.8 mm, vias 0 -> 2
- net Net-(U3-~{CHRG}): track 0.00 -> 32.0 mm, vias 0 -> 2
- net Net-(D5-K): track 0.00 -> 2.23 mm
- net Net-(D4-K): track 0.00 -> 2.13 mm
- net GND: track 18.5 -> 19.5 mm, vias 18 -> 19

Commit message: Correction des erreurs (DRC)
Routing:
- net EPD_DC: track 42.9 -> 44.8 mm
- net GND: vias 19 -> 56

Commit message: Suite DRC
Parts:
- J1: footprint Composants_Perso:Connector_24P_epaper -> Composants_Perso:Connector_1x24_epaper
- moved GDR1 1.60 mm to (126.3, 86.6)
- moved J10 1.28 mm to (192.4, 94.5)
- moved F1 0.17 mm to (191.1, 104.5)
Routing:
- net VBUS: track 73.8 -> 55.1 mm
- net Net-(J10-Pin_2): track 4.12 -> 5.31 mm
- net GDR: track 11.6 -> 12.7 mm
- net GND: vias 56 -> 57

Commit message: pusg
Parts:
- Q5: value FS8205A -> SOP65P640X120-8N
Routing:
- net VBUS: track 55.1 -> 71.3 mm
- net GND: track 19.5 -> 26.5 mm, vias 57 -> 60
- net EPD_BUSY: track 44.6 -> 45.1 mm

Commit message: Placement + routage V3
Parts:
- Q5: value SOP65P640X120-8N -> FS8205A
- moved C21 0.88 mm to (151.3, 68.8)
- moved TP30 0.75 mm to (137.8, 70.4)
- moved D8 0.50 mm to (138.8, 73.7)
- renumbered TP20 to VDD1
Routing:
- net EPD_RST: track 43.3 -> 45.4 mm
- net Net-(J9-Pin_1): track 82.2 -> 84.0 mm
- net EPD_BUSY: track 45.1 -> 46.8 mm
- net EPD_DC: track 44.8 -> 46.2 mm
- net EPD_CS: track 44.5 -> 45.7 mm
- net EPD_SCK: track 44.7 -> 45.6 mm
- net EPD_DIN: track 44.4 -> 45.2 mm
- net Net-(D2-K): track 8.73 -> 9.37 mm
- net GND: track 26.5 -> 25.9 mm, vias 60 -> 62
Other:
- board text added: "Station Météo V1 Maël et Rémi"
