File: Station_Meteo_pcb.kicad_pcb (KiCad board)
At the start: 2 copper layers, 107 x 64 mm, 123 parts, among them J1 ZX-FPC-FWSX0.5PH224, J10 DZ254S-11-02-48, J11 DZ254S-11-02-48, J2 UC18-0B06F68011, J3 BH127VS-14P-H49, J4 DZ254S-11-02-48, J5 DZ254S-11-02-48, J6 DZ254S-11-02-48, J8 DZ254S-11-02-48, J9 DZ254S-11-02-48, Q1 AO3400A, Q2 AO3400A, Q3 AO3401A, Q5 FS8205A, Q6 AO3401A, Q7 AO3401A, Q8 AO3401A, Q9 AO3400A, U1 BME280, U2 STM32L476RGTx, U3 TP4056-42-ESOP8, U4 TPS63802DLAR, U5 DW01A, Y2 Crystal

Commit message: push
Routing:
- net GND: vias 62 -> 63

Commit message: Commande
Routing:
- net GNDA: vias 5 -> 8
- net GND1: vias 6 -> 7
- net GND: vias 63 -> 205
Other:
- board text added: "Station Météo V1 Maël et Rémi 2026"
- board text removed: "Station Météo V1 Maël et Rémi"

Commit message: modif pour commande
Parts:
- C24, C28: value 1u/50 -> 1u/50V
- J4, J5, J6: footprint Connector_PinHeader_2.54mm:PinHeader_1x02_P2.54mm_Vertical_SMD_Pin1Right -> Connector_PinHeader_2.54mm:PinHeader_1x02_P2.54mm_Vertical_SMD_Pin1Left
- moved Q3 1.04 mm to (145.7, 83.3)
- moved R35 1.04 mm to (186.8, 67.6), turned to 180 degrees
- moved J6 0.69 mm to (140.0, 82.7), turned to 180 degrees
- moved J5 0.29 mm to (119.0, 52.1), turned to 180 degrees
- turned J4 to 0 degrees
Routing:
- net Net-(D1-A): track 17.5 -> 19.8 mm
- net +3V3: track 129.9 -> 128.0 mm
- net Net-(Q2-D): track 6.90 -> 6.22 mm
- net ALIM_SCREEN: track 17.2 -> 17.7 mm
- net Net-(J4-Pin_2): track 12.0 -> 11.4 mm

Commit message: last p
Parts:
- Q5: value FS8205A -> FH8205A
